Commit message: enable moveit command

File: indy7_description/urdf/indy7_eye.xacro (robot description, xacro)
@@ -6,5 +6,5 @@
 	<xacro:property name="indy_material" value="metal_grey"/>
 	<!-- <material name="grey"> <color rgba="0.5 0.5 0.5 1"/> </material> -->
-	<link name="ground"/>
+	<link name="world"/>
 	<link name="link0">
 		<visual>
@@ -199,5 +199,5 @@
 	<link name="tcp"/>
 	<joint name="global" type="fixed">
-		<parent link="ground"/>
+		<parent link="world"/>
 		<child link="link0"/>
 		<origin xyz="0 0 0" rpy="0 0 0"/>

File: indyrp2_description/urdf/indyrp2.xacro (robot description, xacro)
@@ -4,5 +4,5 @@
 	<xacro:property name="PI" value="3.1415926535897931"/>
 	<xacro:property name="indy_material" value="metal_grey"/>
-	<link name = "ground" />
+	<link name = "world" />
     <link name = "link0">
         <visual>
@@ -167,5 +167,5 @@
     <link name = "tcp" />
     <joint name = "global" type = "fixed">
-    	<parent link = "ground"/>
+    	<parent link = "world"/>
     	<child link = "link0"/>
     	<origin xyz = "0 0 0" rpy = "0 0 0"/>
