Commit message: add indyeye model

File: indy7_description/urdf/indy7.xacro (robot description, xacro)
@@ -195,39 +195,45 @@
 		<origin xyz="0 0 0" rpy="0 0 0"/>
 	</joint>
-	<joint name="joint0" type="continuous">
+	<joint name="joint0" type="revolute">
 		<parent link="link0"/>
 		<child link="link1"/>
 		<origin xyz="0 0 0.03000000" rpy="0 0 0"/>
 		<axis xyz="0 0 1"/>
-	</joint>
-	<joint name="joint1" type="continuous">
+		<limit effort="10" velocity="1" lower="-${175*PI/180}" upper="${175*PI/180}"/>
+	</joint>
+	<joint name="joint1" type="revolute">
 		<parent link="link1"/>
 		<child link="link2"/>
 		<origin xyz="0 -0.10900000 0.22200000" rpy="${PI/2} ${PI/2} 0"/>
 		<axis xyz="0 0 1"/>
-	</joint>
-	<joint name="joint2" type="continuous">
+		<limit effort="10" velocity="1" lower="-${175*PI/180}" upper="${175*PI/180}"/>
+	</joint>
+	<joint name="joint2" type="revolute">
 		<parent link="link2"/>
 		<child link="link3"/>
 		<origin xyz="-0.45000000 +0.00000000 -0.03050000" rpy="0 0 0"/>
 		<axis xyz="0 0 1"/>
-	</joint>
-	<joint name="joint3" type="continuous">
+		<limit effort="10" velocity="1" lower="-${175*PI/180}" upper="${175*PI/180}"/>
+	</joint>
+	<joint name="joint3" type="revolute">
 		<parent link="link3"/>
 		<child link="link4"/>
 		<origin xyz="-0.26700000 +0.00000000 -0.07500000" rpy="-${PI/2} 0 ${PI/2}"/>
 		<axis xyz="0 0 1"/>
-	</joint>
-	<joint name="joint4" type="continuous">
+		<limit effort="10" velocity="1" lower="-${175*PI/180}" upper="${175*PI/180}"/>
+	</joint>
+	<joint name="joint4" type="revolute">
 		<parent link="link4"/>
 		<child link="link5"/>
 		<origin xyz="+0.00000000 -0.11400000 +0.08300000" rpy="${PI/2} ${PI/2} 0"/>
 		<axis xyz="0 0 1"/>
-	</joint>
-	<joint name="joint5" type="continuous">
+		<limit effort="10" velocity="1" lower="-${175*PI/180}" upper="${175*PI/180}"/>
+	</joint>
+	<joint name="joint5" type="revolute">
 		<parent link="link5"/>
 		<child link="link6"/>
 		<origin xyz="-0.16800000 +0.00000000 +0.06900000" rpy="-${PI/2} 0 ${PI/2}"/>
 		<axis xyz="0 0 1"/>
+		<limit effort="10" velocity="1" lower="-${215*PI/180}" upper="${215*PI/180}"/>
 	</joint>
 	<joint name="tcp" type="fixed">

Commit message: correct inertia

File: indy7_description/urdf/indy7.xacro (robot description, xacro)
@@ -6,5 +6,5 @@
 	<xacro:property name="indy_material" value="metal_grey"/>
 	<!-- <material name="grey"> <color rgba="0.5 0.5 0.5 1"/> </material> -->
-	<link name="ground"/>
+	<link name="world"/>
 	<link name="link0">
 		<visual>
@@ -18,5 +18,5 @@
 			<origin xyz="0 0 0" rpy="0 0 0"/>
 			<geometry>
-				<cylinder length="0.06" radius="0.102"/>
+				<cylinder length="0.075" radius="0.102"/>
 			</geometry>
 		</collision>
@@ -49,5 +49,5 @@
 		<inertial>
 			<origin xyz="0 0 0" rpy="0 0 0"/>
-			<mass value="1.59306955"/>
+			<mass value="11.8030102"/>
 			<inertia ixx="+0.15418559" iyy="+0.12937017" izz="+0.05964415" ixy="-0.00000235" iyz="-0.04854267" ixz="+0.00001739"/>
 		</inertial>
@@ -81,6 +81,6 @@
 		<inertial>
 			<origin xyz="0 0 0" rpy="0 0 0"/>
-			<mass value="0.18"/>
-			<inertia ixx="+0.29356980" iyy="+0.25088420" izz="+0.03620519" ixy="-0.00000040" iyz="+0.03727972" ixz="+0.00001441"/>
+			<mass value="7.99292141"/>
+			<inertia ixx="+0.29356980" iyy="+0.28094142" izz="+0.03620609" ixy="-0.00000040" iyz="+0.03727972" ixz="+0.00001441"/>
 		</inertial>
 	</link>
@@ -107,5 +107,5 @@
 		<inertial>
 			<origin xyz="0 0 0" rpy="0 0 0"/>
-			<mass value="0.18"/>
+			<mass value="2.99134127"/>
 			<inertia ixx="+0.03424593" iyy="+0.03406024" izz="+0.00450477" ixy="+0.00000149" iyz="+0.00186009" ixz="+0.00000724"/>
 		</inertial>
@@ -139,6 +139,6 @@
 		<inertial>
 			<origin xyz="0 0 0" rpy="0 0 0"/>
-			<mass value="0.18"/>
-			<inertia ixx="+0.00670405" iyy="+0.00670405" izz="+0.00617624" ixy="+0.00000375" iyz="-0.00127967" ixz="+0.00000150"/>
+			<mass value="2.12317035"/>
+			<inertia ixx="+0.00670405" iyy="+0.00279246" izz="+0.00619341" ixy="+0.00000375" iyz="-0.00127967" ixz="+0.00000150"/>
 		</inertial>
 	</link>
@@ -165,5 +165,5 @@
 		<inertial>
 			<origin xyz="0 0 0" rpy="0 0 0"/>
-			<mass value="0.18"/>
+			<mass value="2.28865091"/>
 			<inertia ixx="+0.00994891" iyy="+0.00978189" izz="+0.00271492" ixy="+0.00000014" iyz="-0.00093546" ixz="+0.00000321"/>
 		</inertial>
@@ -185,5 +185,5 @@
 		<inertial>
 			<origin xyz="0 0 0" rpy="0 0 0"/>
-			<mass value="0.18"/>
+			<mass value="0.40083918"/>
 			<inertia ixx="0.00043534" iyy="0.00044549" izz="0.00059634" ixy="+0.00000013" iyz="+0.00000051" ixz="-0.00000002"/>
 		</inertial>
@@ -191,5 +191,5 @@
 	<link name="tcp"/>
 	<joint name="global" type="fixed">
-		<parent link="ground"/>
+		<parent link="world"/>
 		<child link="link0"/>
 		<origin xyz="0 0 0" rpy="0 0 0"/>
@@ -198,5 +198,5 @@
 		<parent link="link0"/>
 		<child link="link1"/>
-		<origin xyz="0 0 0.03000000" rpy="0 0 0"/>
+		<origin xyz="0 0 0.0775" rpy="0 0 0"/>
 		<axis xyz="0 0 1"/>
 		<limit effort="10" velocity="1" lower="-${175*PI/180}" upper="${175*PI/180}"/>

Commit message: ;

File: indy7_description/urdf/indy7.xacro (robot description, xacro)
@@ -6,5 +6,4 @@
 	<xacro:property name="indy_material" value="metal_grey"/>
 	<!-- <material name="grey"> <color rgba="0.5 0.5 0.5 1"/> </material> -->
-	<link name="world"/>
 	<link name="link0">
 		<visual>
@@ -190,9 +189,4 @@
 	</link>
 	<link name="tcp"/>
-	<joint name="global" type="fixed">
-		<parent link="world"/>
-		<child link="link0"/>
-		<origin xyz="0 0 0" rpy="0 0 0"/>
-	</joint>
 	<joint name="joint0" type="revolute">
 		<parent link="link0"/>

File: indy7_description/urdf/indy7_eye.xacro (robot description, xacro)
@@ -5,6 +5,4 @@
 	<xacro:property name="PI" value="3.1415926535897931"/>
 	<xacro:property name="indy_material" value="metal_grey"/>
-	<!-- <material name="grey"> <color rgba="0.5 0.5 0.5 1"/> </material> -->
-	<link name="world"/>
 	<link name="link0">
 		<visual>
@@ -198,9 +196,4 @@
 	</link>
 	<link name="tcp"/>
-	<joint name="global" type="fixed">
-		<parent link="world"/>
-		<child link="link0"/>
-		<origin xyz="0 0 0" rpy="0 0 0"/>
-	</joint>
 	<joint name="joint0" type="revolute">
 		<parent link="link0"/>

Commit message: bugfix for noetic

File: indy7_description/urdf/indy7.xacro (robot description, xacro)
@@ -239,8 +239,8 @@
 		<type>transmission_interface/SimpleTransmission</type>
 		<joint name="joint0">
-			<hardwareInterface>PositionJointInterface</hardwareInterface>
+			<hardwareInterface>hardware_interface/PositionJointInterface</hardwareInterface>
 		</joint>
 		<actuator name="motor0">
-			<hardwareInterface>PositionJointInterface</hardwareInterface>
+			<hardwareInterface>hardware_interface/PositionJointInterface</hardwareInterface>
 			<mechanicalReduction>1</mechanicalReduction>
 		</actuator>
@@ -249,8 +249,8 @@
 		<type>transmission_interface/SimpleTransmission</type>
 		<joint name="joint1">
-			<hardwareInterface>PositionJointInterface</hardwareInterface>
+			<hardwareInterface>hardware_interface/PositionJointInterface</hardwareInterface>
 		</joint>
 		<actuator name="motor1">
-			<hardwareInterface>PositionJointInterface</hardwareInterface>
+			<hardwareInterface>hardware_interface/PositionJointInterface</hardwareInterface>
 			<mechanicalReduction>1</mechanicalReduction>
 		</actuator>
@@ -259,8 +259,8 @@
 		<type>transmission_interface/SimpleTransmission</type>
 		<joint name="joint2">
-			<hardwareInterface>PositionJointInterface</hardwareInterface>
+			<hardwareInterface>hardware_interface/PositionJointInterface</hardwareInterface>
 		</joint>
 		<actuator name="motor2">
-			<hardwareInterface>PositionJointInterface</hardwareInterface>
+			<hardwareInterface>hardware_interface/PositionJointInterface</hardwareInterface>
 			<mechanicalReduction>1</mechanicalReduction>
 		</actuator>
@@ -269,8 +269,8 @@
 		<type>transmission_interface/SimpleTransmission</type>
 		<joint name="joint3">
-			<hardwareInterface>PositionJointInterface</hardwareInterface>
+			<hardwareInterface>hardware_interface/PositionJointInterface</hardwareInterface>
 		</joint>
 		<actuator name="motor3">
-			<hardwareInterface>PositionJointInterface</hardwareInterface>
+			<hardwareInterface>hardware_interface/PositionJointInterface</hardwareInterface>
 			<mechanicalReduction>1</mechanicalReduction>
 		</actuator>
@@ -279,8 +279,8 @@
 		<type>transmission_interface/SimpleTransmission</type>
 		<joint name="joint4">
-			<hardwareInterface>PositionJointInterface</hardwareInterface>
+			<hardwareInterface>hardware_interface/PositionJointInterface</hardwareInterface>
 		</joint>
 		<actuator name="motor4">
-			<hardwareInterface>PositionJointInterface</hardwareInterface>
+			<hardwareInterface>hardware_interface/PositionJointInterface</hardwareInterface>
 			<mechanicalReduction>1</mechanicalReduction>
 		</actuator>
@@ -289,8 +289,8 @@
 		<type>transmission_interface/SimpleTransmission</type>
 		<joint name="joint5">
-			<hardwareInterface>PositionJointInterface</hardwareInterface>
+			<hardwareInterface>hardware_interface/PositionJointInterface</hardwareInterface>
 		</joint>
 		<actuator name="motor5">
-			<hardwareInterface>PositionJointInterface</hardwareInterface>
+			<hardwareInterface>hardware_interface/PositionJointInterface</hardwareInterface>
 			<mechanicalReduction>1</mechanicalReduction>
 		</actuator>

File: indy7_description/urdf/indy7_fixed.xacro (robot description, xacro)
@@ -6,5 +6,5 @@
 		<parent link="world"/>
 		<child link="link0"/>
-		<origin xyz="0 0 0" rpy="0 0 0"/>
+		<origin xyz="0 0 0.1" rpy="0 0 0"/>
 	</joint>
 </robot>

Commit message: Update indy7.xacro

File: indy7_description/urdf/indy7.xacro (robot description, xacro)
@@ -17,5 +17,6 @@
 			<origin xyz="0 0 0" rpy="0 0 0"/>
 			<geometry>
-				<cylinder length="0.075" radius="0.102"/>
+				<mesh filename="package://indy7_description/meshes/stl/Indy7_0.stl"/>
+				<!--<cylinder length="0.075" radius="0.102"/>-->
 			</geometry>
 		</collision>

Commit message: 1130

File: indy7_description/urdf/indy7.xacro (robot description, xacro)
@@ -15,5 +15,5 @@
 		</visual>
 		<collision>
-			<origin xyz="0 0 0" rpy="0 0 0"/>
+			<origin xyz="0 0 0.0375" rpy="0 0 0"/>
 			<geometry>
 				<cylinder length="0.075" radius="0.102"/>
@@ -194,5 +194,5 @@
 		<origin xyz="0 0 0.0775" rpy="0 0 0"/>
 		<axis xyz="0 0 1"/>
-		<limit effort="10" velocity="1" lower="-${175*PI/180}" upper="${175*PI/180}"/>
+		<limit effort="200" velocity="1" lower="-${175*PI/180}" upper="${175*PI/180}"/>
 	</joint>
 	<joint name="joint1" type="revolute">
@@ -201,5 +201,5 @@
 		<origin xyz="0 -0.10900000 0.22200000" rpy="${PI/2} ${PI/2} 0"/>
 		<axis xyz="0 0 1"/>
-		<limit effort="10" velocity="1" lower="-${175*PI/180}" upper="${175*PI/180}"/>
+		<limit effort="200" velocity="1" lower="-${175*PI/180}" upper="${175*PI/180}"/>
 	</joint>
 	<joint name="joint2" type="revolute">
@@ -208,5 +208,5 @@
 		<origin xyz="-0.45000000 +0.00000000 -0.03050000" rpy="0 0 0"/>
 		<axis xyz="0 0 1"/>
-		<limit effort="10" velocity="1" lower="-${175*PI/180}" upper="${175*PI/180}"/>
+		<limit effort="200" velocity="1" lower="-${175*PI/180}" upper="${175*PI/180}"/>
 	</joint>
 	<joint name="joint3" type="revolute">

File: indy7_description/urdf/indy7_fixed.xacro (robot description, xacro)
@@ -6,5 +6,11 @@
 		<parent link="world"/>
 		<child link="link0"/>
-		<origin xyz="0 0 0.1" rpy="0 0 0"/>
+		<origin xyz="0 0 0.0" rpy="0 0 0"/>
 	</joint>
+    <!-- Import macro for realsense-RS200 camera-->
+    <xacro:include filename="$(find realsense_gazebo_plugin)/urdf/realsense-RS200.macro.xacro"/>
+    <!-- Create camera instance -->
+    <xacro:realsense-rs200 prefix="" parent="tcp">
+    <origin rpy="0 -1.5707 0 " xyz="-0.05 0 0.05"/>
+    </xacro:realsense-rs200>
 </robot>

Commit message: asdf

File: indy7_description/urdf/indy7.xacro (robot description, xacro)
@@ -215,5 +215,5 @@
 		<origin xyz="-0.26700000 +0.00000000 -0.07500000" rpy="-${PI/2} 0 ${PI/2}"/>
 		<axis xyz="0 0 1"/>
-		<limit effort="10" velocity="1" lower="-${175*PI/180}" upper="${175*PI/180}"/>
+		<limit effort="100" velocity="1" lower="-${175*PI/180}" upper="${175*PI/180}"/>
 	</joint>
 	<joint name="joint4" type="revolute">
@@ -229,5 +229,5 @@
 		<origin xyz="-0.16800000 +0.00000000 +0.06900000" rpy="-${PI/2} 0 ${PI/2}"/>
 		<axis xyz="0 0 1"/>
-		<limit effort="10" velocity="1" lower="-${215*PI/180}" upper="${215*PI/180}"/>
+		<limit effort="10" velocity="1" lower="${-PI}" upper="${PI}"/>
 	</joint>
 	<joint name="tcp" type="fixed">

Commit message: update physical parameters

File: indy7_description/urdf/indy7.xacro (robot description, xacro)
@@ -22,6 +22,6 @@
 		<inertial>
 			<origin xyz="0 0 0" rpy="0 0 0"/>
-			<mass value="1.59306955"/>
-			<inertia ixx="+0.00572623" iyy="+0.00558959" izz="+0.00966674" ixy="+0.00000251" iyz="-0.00000014" ixz="-0.00011380"/>
+			<mass value="1.67030785"/>
+			<inertia ixx="+0.00661309" iyy="+0.00644765" izz="+0.00792090" ixy="+0.00000183" iyz="-0.00000027" ixz="+0.00002695"/>
 		</inertial>
 	</link>
@@ -48,6 +48,6 @@
 		<inertial>
 			<origin xyz="0 0 0" rpy="0 0 0"/>
-			<mass value="11.8030102"/>
-			<inertia ixx="+0.15418559" iyy="+0.12937017" izz="+0.05964415" ixy="-0.00000235" iyz="-0.04854267" ixz="+0.00001739"/>
+			<mass value="11.44444535"/>
+			<inertia ixx="+0.35065005" iyy="+0.30479800" izz="+0.06003147" ixy="+0.00011931" iyz="-0.10984447" ixz="-0.00037553"/>
 		</inertial>
 	</link>
@@ -80,6 +80,6 @@
 		<inertial>
 			<origin xyz="0 0 0" rpy="0 0 0"/>
-			<mass value="7.99292141"/>
-			<inertia ixx="+0.29356980" iyy="+0.28094142" izz="+0.03620609" ixy="-0.00000040" iyz="+0.03727972" ixz="+0.00001441"/>
+			<mass value="5.84766553"/>
+			<inertia ixx="+0.03599743" iyy="+0.72293306" izz="+0.70024119" ixy="-0.00004693" iyz="+0.00000176" ixz="-0.05240346"/>
 		</inertial>
 	</link>
@@ -106,6 +106,6 @@
 		<inertial>
 			<origin xyz="0 0 0" rpy="0 0 0"/>
-			<mass value="2.99134127"/>
-			<inertia ixx="+0.03424593" iyy="+0.03406024" izz="+0.00450477" ixy="+0.00000149" iyz="+0.00186009" ixz="+0.00000724"/>
+			<mass value="2.68206064"/>
+			<inertia ixx="+0.01617210" iyy="+0.11364055" izz="+0.10022522" ixy="-0.00011817" iyz="-0.00004371" ixz="+0.03341882"/>
 		</inertial>
 	</link>
@@ -138,6 +138,6 @@
 		<inertial>
 			<origin xyz="0 0 0" rpy="0 0 0"/>
-			<mass value="2.12317035"/>
-			<inertia ixx="+0.00670405" iyy="+0.00279246" izz="+0.00619341" ixy="+0.00000375" iyz="-0.00127967" ixz="+0.00000150"/>
+			<mass value="2.12987371"/>
+			<inertia ixx="+0.02798891" iyy="+0.01443076" izz="+0.01496211" ixy="+0.00003893" iyz="-0.01266296" ixz="-0.00004768"/>
 		</inertial>
 	</link>
@@ -164,6 +164,6 @@
 		<inertial>
 			<origin xyz="0 0 0" rpy="0 0 0"/>
-			<mass value="2.28865091"/>
-			<inertia ixx="+0.00994891" iyy="+0.00978189" izz="+0.00271492" ixy="+0.00000014" iyz="-0.00093546" ixz="+0.00000321"/>
+			<mass value="2.22412271"/>
+			<inertia ixx="+0.01105297" iyy="+0.03698291" izz="+0.02754795" ixy="+0.00005517" iyz="-0.00003740" ixz="-0.01481977"/>
 		</inertial>
 	</link>
@@ -184,6 +184,6 @@
 		<inertial>
 			<origin xyz="0 0 0" rpy="0 0 0"/>
-			<mass value="0.40083918"/>
-			<inertia ixx="0.00043534" iyy="0.00044549" izz="0.00059634" ixy="+0.00000013" iyz="+0.00000051" ixz="-0.00000002"/>
+			<mass value="0.38254932"/>
+			<inertia ixx="+0.00078982" iyy="+0.00079764" izz="+0.00058319" ixy="-0.00000034" iyz="-0.00000508" ixz="+0.00000083"/>
 		</inertial>
 	</link>

File: indy7_description/urdf/indy7_eye.xacro (robot description, xacro)
@@ -21,6 +21,6 @@
 		<inertial>
 			<origin xyz="0 0 0" rpy="0 0 0"/>
-			<mass value="1.59306955"/>
-			<inertia ixx="+0.00572623" iyy="+0.00558959" izz="+0.00966674" ixy="+0.00000251" iyz="-0.00000014" ixz="-0.00011380"/>
+			<mass value="1.67030785"/>
+			<inertia ixx="+0.00661309" iyy="+0.00644765" izz="+0.00792090" ixy="+0.00000183" iyz="-0.00000027" ixz="+0.00002695"/>
 		</inertial>
 	</link>
@@ -47,6 +47,6 @@
 		<inertial>
 			<origin xyz="0 0 0" rpy="0 0 0"/>
-			<mass value="1.59306955"/>
-			<inertia ixx="+0.15418559" iyy="+0.12937017" izz="+0.05964415" ixy="-0.00000235" iyz="-0.04854267" ixz="+0.00001739"/>
+			<mass value="11.44444535"/>
+			<inertia ixx="+0.35065005" iyy="+0.30479800" izz="+0.06003147" ixy="+0.00011931" iyz="-0.10984447" ixz="-0.00037553"/>
 		</inertial>
 	</link>
@@ -79,7 +79,6 @@
 		<inertial>
 			<origin xyz="0 0 0" rpy="0 0 0"/>
-			<mass value="0.18"/>
-			<inertia ixx="+0.29356980" iyy="+0.25088420" izz="+0.03620519" ixy="-0.00000040" iyz="+0.03727972" ixz="+0.00001441"/>
-		</inertial>
+			<mass value="5.84766553"/>
+			<inertia ixx="+0.03599743" iyy="+0.72293306" izz="+0.70024119" ixy="-0.00004693" iyz="+0.00000176" ixz="-0.05240346"/>		</inertial>
 	</link>
 	<link name="link3">
@@ -105,6 +104,6 @@
 		<inertial>
 			<origin xyz="0 0 0" rpy="0 0 0"/>
-			<mass value="0.18"/>
-			<inertia ixx="+0.03424593" iyy="+0.03406024" izz="+0.00450477" ixy="+0.00000149" iyz="+0.00186009" ixz="+0.00000724"/>
+			<mass value="2.68206064"/>
+			<inertia ixx="+0.01617210" iyy="+0.11364055" izz="+0.10022522" ixy="-0.00011817" iyz="-0.00004371" ixz="+0.03341882"/>
 		</inertial>
 	</link>
@@ -137,6 +136,6 @@
 		<inertial>
 			<origin xyz="0 0 0" rpy="0 0 0"/>
-			<mass value="0.18"/>
-			<inertia ixx="+0.00670405" iyy="+0.00670405" izz="+0.00617624" ixy="+0.00000375" iyz="-0.00127967" ixz="+0.00000150"/>
+			<mass value="2.12987371"/>
+			<inertia ixx="+0.02798891" iyy="+0.01443076" izz="+0.01496211" ixy="+0.00003893" iyz="-0.01266296" ixz="-0.00004768"/>
 		</inertial>
 	</link>
@@ -163,6 +162,6 @@
 		<inertial>
 			<origin xyz="0 0 0" rpy="0 0 0"/>
-			<mass value="0.18"/>
-			<inertia ixx="+0.00994891" iyy="+0.00978189" izz="+0.00271492" ixy="+0.00000014" iyz="-0.00093546" ixz="+0.00000321"/>
+			<mass value="2.22412271"/>
+			<inertia ixx="+0.01105297" iyy="+0.03698291" izz="+0.02754795" ixy="+0.00005517" iyz="-0.00003740" ixz="-0.01481977"/>
 		</inertial>
 	</link>
@@ -183,6 +182,6 @@
 		<inertial>
 			<origin xyz="0 0 0" rpy="0 0 0"/>
-			<mass value="0.18"/>
-			<inertia ixx="0.00043534" iyy="0.00044549" izz="0.00059634" ixy="+0.00000013" iyz="+0.00000051" ixz="-0.00000002"/>
+			<mass value="0.38254932"/>
+			<inertia ixx="+0.00078982" iyy="+0.00079764" izz="+0.00058319" ixy="-0.00000034" iyz="-0.00000508" ixz="+0.00000083"/>
 		</inertial>
 	</link>

File: indyrp2_description/urdf/indyrp2.xacro (robot description, xacro)
@@ -21,6 +21,6 @@
          <inertial>
             <origin xyz="0 0 0" rpy="0 0 0"/>
-            <mass value="5.44309" />
-            <inertia ixx="0.0236" iyy="0.0234" izz="0.0137" ixy="0" iyz="0.0001" ixz="0"/>
+			<mass value="1.67030785"/>
+			<inertia ixx="+0.00661309" iyy="+0.00644765" izz="+0.00792090" ixy="+0.00000183" iyz="-0.00000027" ixz="+0.00002695"/>
         </inertial>
     </link>
@@ -41,6 +41,6 @@
          <inertial>
             <origin xyz="0 0 0" rpy="0 0 0"/>
-            <mass value="5.50328" />
-            <inertia ixx="0.0227" iyy="0.0121" izz="0.0212" ixy="0" iyz="0.0013" ixz="0" />
+			<mass value="11.44444535"/>
+			<inertia ixx="+0.35065005" iyy="+0.30479800" izz="+0.06003147" ixy="+0.00011931" iyz="-0.10984447" ixz="-0.00037553"/>
         </inertial>
     </link>
@@ -61,6 +61,6 @@
          <inertial>
             <origin xyz="0 0 0" rpy="0 0 0"/>
-            <mass value="5.95397" />
-            <inertia ixx="0.1175" iyy="0.1172" izz="0.0131" ixy="00" iyz="0.0037" ixz="0"/>
+            <mass value="4.43308185" />
+            <inertia ixx="+0.03742681" iyy="+0.32119654" izz="+0.29396155" ixy="-0.00003176" iyz="-0.00000808" ixz="+0.07906734"/>
         </inertial>
     </link>
@@ -81,6 +81,6 @@
          <inertial>
             <origin xyz="0 0 0" rpy="0 0 0"/>
-            <mass value="4.08259" />
-            <inertia ixx="0.0132" iyy="0.0068" izz="0.0125" ixy="0" iyz="-0.0008" ixz="0"/>
+            <mass value="2.87045928" />
+            <inertia ixx="+0.04098160" iyy="+0.02106773" izz="+0.02277477" ixy="+0.00000747" iyz="-0.01817157" ixz="-0.00000916"/>
         </inertial>
     </link>
@@ -101,6 +101,6 @@
          <inertial>
             <origin xyz="0 0 0" rpy="0 0 0"/>
-            <mass value="4.02733" />
-            <inertia ixx="0.0674" iyy="0.067" izz="0.0071" ixy="0" iyz="-0.0027" ixz="0"/>
+			<mass value="2.68206064"/>
+			<inertia ixx="+0.01617210" iyy="+0.11364055" izz="+0.10022522" ixy="-0.00011817" iyz="-0.00004371" ixz="+0.03341882"/>
         </inertial>
     </link>
@@ -121,6 +121,6 @@
          <inertial>
             <origin xyz="0 0 0" rpy="0 0 0"/>
-            <mass value="2.52863" />
-            <inertia ixx="0.0066" iyy="0.0033" izz="0.0062" ixy="0" iyz="0.0003" ixz="0"/>
+			<mass value="2.12987371"/>
+			<inertia ixx="+0.02798891" iyy="+0.01443076" izz="+0.01496211" ixy="+0.00003893" iyz="-0.01266296" ixz="-0.00004768"/>
         </inertial>
     </link>
@@ -141,6 +141,6 @@
          <inertial>
             <origin xyz="0 0 0" rpy="0 0 0"/>
-            <mass value="2.03152" />
-            <inertia ixx="0.0042" iyy="0.0041" izz="0.0018" ixy="0" iyz="0.0003" ixz="0"/>
+			<mass value="2.22412271"/>
+			<inertia ixx="+0.01105297" iyy="+0.03698291" izz="+0.02754795" ixy="+0.00005517" iyz="-0.00003740" ixz="-0.01481977"/>
         </inertial>
     </link>
@@ -161,6 +161,6 @@
          <inertial>
             <origin xyz="0 0 0" rpy="0 0 0"/>
-            <mass value="0.17194" />
-            <inertia ixx="0.0001" iyy="0.0001" izz="0.0001" ixy="0" iyz="0" ixz="0"/>
+			<mass value="0.38254932"/>
+			<inertia ixx="+0.00078982" iyy="+0.00079764" izz="+0.00058319" ixy="-0.00000034" iyz="-0.00000508" ixz="+0.00000083"/>
         </inertial>
     </link>
