Commit message: update physical parameters -add COM, Camera dynamics

File: indy7_description/urdf/indy7.xacro (robot description, xacro)
@@ -21,5 +21,5 @@
 		</collision>
 		<inertial>
-			<origin xyz="0 0 0" rpy="0 0 0"/>
+			<origin xyz="0.00131966 -0.00000218 0.03212832" rpy="0 0 0"/>
 			<mass value="1.67030785"/>
 			<inertia ixx="+0.00661309" iyy="+0.00644765" izz="+0.00792090" ixy="+0.00000183" iyz="-0.00000027" ixz="+0.00002695"/>
@@ -47,5 +47,5 @@
 		</collision>
 		<inertial>
-			<origin xyz="0 0 0" rpy="0 0 0"/>
+			<origin xyz="-0.00023749 -0.04310313 0.13245396" rpy="0 0 0"/>
 			<mass value="11.44444535"/>
 			<inertia ixx="+0.35065005" iyy="+0.30479800" izz="+0.06003147" ixy="+0.00011931" iyz="-0.10984447" ixz="-0.00037553"/>
@@ -79,5 +79,5 @@
 		</collision>
 		<inertial>
-			<origin xyz="0 0 0" rpy="0 0 0"/>
+			<origin xyz="-0.29477536 -0.00002361 0.04762554" rpy="0 0 0"/>
 			<mass value="5.84766553"/>
 			<inertia ixx="+0.03599743" iyy="+0.72293306" izz="+0.70024119" ixy="-0.00004693" iyz="+0.00000176" ixz="-0.05240346"/>
@@ -105,5 +105,5 @@
 		</collision>
 		<inertial>
-			<origin xyz="0 0 0" rpy="0 0 0"/>
+			<origin xyz="-0.16804016 0.00021421 -0.07000383" rpy="0 0 0"/>
 			<mass value="2.68206064"/>
 			<inertia ixx="+0.01617210" iyy="+0.11364055" izz="+0.10022522" ixy="-0.00011817" iyz="-0.00004371" ixz="+0.03341882"/>
@@ -137,5 +137,5 @@
 		</collision>
 		<inertial>
-			<origin xyz="0 0 0" rpy="0 0 0"/>
+			<origin xyz="-0.00026847 -0.07098440 0.07649128" rpy="0 0 0"/>
 			<mass value="2.12987371"/>
 			<inertia ixx="+0.02798891" iyy="+0.01443076" izz="+0.01496211" ixy="+0.00003893" iyz="-0.01266296" ixz="-0.00004768"/>
@@ -163,5 +163,5 @@
 		</collision>
 		<inertial>
-			<origin xyz="0 0 0" rpy="0 0 0"/>
+			<origin xyz="-0.09796232 -0.00023114 0.06445892" rpy="0 0 0"/>
 			<mass value="2.22412271"/>
 			<inertia ixx="+0.01105297" iyy="+0.03698291" izz="+0.02754795" ixy="+0.00005517" iyz="-0.00003740" ixz="-0.01481977"/>
@@ -183,5 +183,5 @@
 		</collision>
 		<inertial>
-			<origin xyz="0 0 0" rpy="0 0 0"/>
+			<origin xyz="0.00008147 -0.00046556 0.03079097" rpy="0 0 0"/>
 			<mass value="0.38254932"/>
 			<inertia ixx="+0.00078982" iyy="+0.00079764" izz="+0.00058319" ixy="-0.00000034" iyz="-0.00000508" ixz="+0.00000083"/>

File: indy7_description/urdf/indy7_eye.xacro (robot description, xacro)
@@ -20,5 +20,5 @@
 		</collision>
 		<inertial>
-			<origin xyz="0 0 0" rpy="0 0 0"/>
+			<origin xyz="0.00131966 -0.00000218 0.03212832" rpy="0 0 0"/>
 			<mass value="1.67030785"/>
 			<inertia ixx="+0.00661309" iyy="+0.00644765" izz="+0.00792090" ixy="+0.00000183" iyz="-0.00000027" ixz="+0.00002695"/>
@@ -46,5 +46,5 @@
 		</collision>
 		<inertial>
-			<origin xyz="0 0 0" rpy="0 0 0"/>
+			<origin xyz="-0.00023749 -0.04310313 0.13245396" rpy="0 0 0"/>
 			<mass value="11.44444535"/>
 			<inertia ixx="+0.35065005" iyy="+0.30479800" izz="+0.06003147" ixy="+0.00011931" iyz="-0.10984447" ixz="-0.00037553"/>
@@ -78,5 +78,5 @@
 		</collision>
 		<inertial>
-			<origin xyz="0 0 0" rpy="0 0 0"/>
+			<origin xyz="-0.29477536 -0.00002361 0.04762554" rpy="0 0 0"/>
 			<mass value="5.84766553"/>
 			<inertia ixx="+0.03599743" iyy="+0.72293306" izz="+0.70024119" ixy="-0.00004693" iyz="+0.00000176" ixz="-0.05240346"/>		</inertial>
@@ -103,5 +103,5 @@
 		</collision>
 		<inertial>
-			<origin xyz="0 0 0" rpy="0 0 0"/>
+			<origin xyz="-0.16804016 0.00021421 -0.07000383" rpy="0 0 0"/>
 			<mass value="2.68206064"/>
 			<inertia ixx="+0.01617210" iyy="+0.11364055" izz="+0.10022522" ixy="-0.00011817" iyz="-0.00004371" ixz="+0.03341882"/>
@@ -135,5 +135,5 @@
 		</collision>
 		<inertial>
-			<origin xyz="0 0 0" rpy="0 0 0"/>
+			<origin xyz="-0.00026847 -0.07098440 0.07649128" rpy="0 0 0"/>
 			<mass value="2.12987371"/>
 			<inertia ixx="+0.02798891" iyy="+0.01443076" izz="+0.01496211" ixy="+0.00003893" iyz="-0.01266296" ixz="-0.00004768"/>
@@ -161,5 +161,5 @@
 		</collision>
 		<inertial>
-			<origin xyz="0 0 0" rpy="0 0 0"/>
+			<origin xyz="-0.09796232 -0.00023114 0.06445892" rpy="0 0 0"/>
 			<mass value="2.22412271"/>
 			<inertia ixx="+0.01105297" iyy="+0.03698291" izz="+0.02754795" ixy="+0.00005517" iyz="-0.00003740" ixz="-0.01481977"/>
@@ -181,5 +181,5 @@
 		</collision>
 		<inertial>
-			<origin xyz="0 0 0" rpy="0 0 0"/>
+			<origin xyz="0.00008147 -0.00046556 0.03079097" rpy="0 0 0"/>
 			<mass value="0.38254932"/>
 			<inertia ixx="+0.00078982" iyy="+0.00079764" izz="+0.00058319" ixy="-0.00000034" iyz="-0.00000508" ixz="+0.00000083"/>
@@ -193,4 +193,9 @@
 			</geometry>
 		</collision>
+		<inertial>
+			<origin xyz="-0.03367995 0.00000829 0.02927357" rpy="0 0 0"/>
+			<mass value="0.75567713"/>
+			<inertia ixx="+0.00139931" iyy="+0.00339558" izz="+0.00283846" ixy="+0.00000029" iyz="+0.00000046" ixz="-0.00052678"/>
+		</inertial>
 	</link>
 	<link name="tcp"/>

File: indyrp2_description/urdf/indyrp2.xacro (robot description, xacro)
@@ -20,5 +20,5 @@
         </collision>
          <inertial>
-            <origin xyz="0 0 0" rpy="0 0 0"/>
+            <origin xyz="0.00131966 -0.00000218 0.03212832" rpy="0 0 0"/>
 			<mass value="1.67030785"/>
 			<inertia ixx="+0.00661309" iyy="+0.00644765" izz="+0.00792090" ixy="+0.00000183" iyz="-0.00000027" ixz="+0.00002695"/>
@@ -40,5 +40,5 @@
         </collision>
          <inertial>
-            <origin xyz="0 0 0" rpy="0 0 0"/>
+            <origin xyz="-0.00023749 -0.04310313 0.13245396" rpy="0 0 0"/>
 			<mass value="11.44444535"/>
 			<inertia ixx="+0.35065005" iyy="+0.30479800" izz="+0.06003147" ixy="+0.00011931" iyz="-0.10984447" ixz="-0.00037553"/>
@@ -60,5 +60,5 @@
         </collision>
          <inertial>
-            <origin xyz="0 0 0" rpy="0 0 0"/>
+            <origin xyz="-0.19234403 0.05941510 0.15292668" rpy="0 0 0"/>
             <mass value="4.43308185" />
             <inertia ixx="+0.03742681" iyy="+0.32119654" izz="+0.29396155" ixy="-0.00003176" iyz="-0.00000808" ixz="+0.07906734"/>
@@ -80,5 +80,5 @@
         </collision>
          <inertial>
-            <origin xyz="0 0 0" rpy="0 0 0"/>
+            <origin xyz="-0.60631468 0.12700778 0.02546394" rpy="0 0 0"/>
             <mass value="2.87045928" />
             <inertia ixx="+0.04098160" iyy="+0.02106773" izz="+0.02277477" ixy="+0.00000747" iyz="-0.01817157" ixz="-0.00000916"/>
@@ -100,5 +100,5 @@
         </collision>
          <inertial>
-            <origin xyz="0 0 0" rpy="0 0 0"/>
+            <origin xyz="-0.16804016 0.00021421 -0.07000383" rpy="0 0 0"/>
 			<mass value="2.68206064"/>
 			<inertia ixx="+0.01617210" iyy="+0.11364055" izz="+0.10022522" ixy="-0.00011817" iyz="-0.00004371" ixz="+0.03341882"/>
@@ -120,5 +120,5 @@
         </collision>
          <inertial>
-            <origin xyz="0 0 0" rpy="0 0 0"/>
+            <origin xyz="-0.00026847 -0.07098440 0.07649128" rpy="0 0 0"/>
 			<mass value="2.12987371"/>
 			<inertia ixx="+0.02798891" iyy="+0.01443076" izz="+0.01496211" ixy="+0.00003893" iyz="-0.01266296" ixz="-0.00004768"/>
@@ -140,5 +140,5 @@
         </collision>
          <inertial>
-            <origin xyz="0 0 0" rpy="0 0 0"/>
+            <origin xyz="-0.09796232 -0.00023114 0.06445892" rpy="0 0 0"/>
 			<mass value="2.22412271"/>
 			<inertia ixx="+0.01105297" iyy="+0.03698291" izz="+0.02754795" ixy="+0.00005517" iyz="-0.00003740" ixz="-0.01481977"/>
@@ -160,5 +160,5 @@
         </collision>
          <inertial>
-            <origin xyz="0 0 0" rpy="0 0 0"/>
+            <origin xyz="0.00008147 -0.00046556 0.03079097" rpy="0 0 0"/>
 			<mass value="0.38254932"/>
 			<inertia ixx="+0.00078982" iyy="+0.00079764" izz="+0.00058319" ixy="-0.00000034" iyz="-0.00000508" ixz="+0.00000083"/>

Commit message: update physical parameters - add 7v2, 12, 12v2 rpv2 urdf.xacro (include dynamics and kinematics, joint limit)

File: indy7_description/urdf/indy7.xacro (robot description, xacro)
@@ -14,10 +14,10 @@
 			<material name="${indy_material}"/>
 		</visual>
-		<collision>
-			<origin xyz="0 0 0" rpy="0 0 0"/>
-			<geometry>
-				<cylinder length="0.075" radius="0.102"/>
-			</geometry>
-		</collision>
+         <collision>
+            <origin xyz="0 0 0" rpy="0 0 0"/>
+           	<geometry>
+				<mesh filename="package://indy7_description/meshes/collision/Indy7_0.stl"/>
+			</geometry>
+        </collision>
 		<inertial>
 			<origin xyz="0.00131966 -0.00000218 0.03212832" rpy="0 0 0"/>
@@ -34,16 +34,10 @@
 			<material name="${indy_material}"/>
 		</visual>
-		<collision>
-			<origin xyz="0 0 0.111" rpy="0 0 0"/>
-			<geometry>
-				<cylinder length="0.222" radius="0.075"/>
-			</geometry>
-		</collision>
-		<collision>
-			<origin xyz="0 -0.0545 0.222" rpy="${PI/2} 0 0"/>
-			<geometry>
-				<cylinder length="0.109" radius="0.075"/>
-			</geometry>
-		</collision>
+         <collision>
+            <origin xyz="0 0 0" rpy="0 0 0"/>
+           	<geometry>
+				<mesh filename="package://indy7_description/meshes/collision/Indy7_1.stl"/>
+			</geometry>
+        </collision>
 		<inertial>
 			<origin xyz="-0.00023749 -0.04310313 0.13245396" rpy="0 0 0"/>
@@ -60,22 +54,10 @@
 			<material name="${indy_material}"/>
 		</visual>
-		<collision>
-			<origin xyz="-0.225 0 0.09" rpy="${PI/2} 0 -${PI/2}"/>
-			<geometry>
-				<cylinder length="0.450" radius="0.063"/>
-			</geometry>
-		</collision>
-		<collision>
-			<origin xyz="0 0 0.045" rpy="0 0 0"/>
-			<geometry>
-				<cylinder length="0.09" radius="0.075"/>
-			</geometry>
-		</collision>
-		<collision>
-			<origin xyz="-0.45 0 0.02975 " rpy="0 0 0"/>
-			<geometry>
-				<cylinder length="0.1205" radius="0.045"/>
-			</geometry>
-		</collision>
+         <collision>
+            <origin xyz="0 0 0" rpy="0 0 0"/>
+           	<geometry>
+				<mesh filename="package://indy7_description/meshes/collision/Indy7_2.stl"/>
+			</geometry>
+        </collision>
 		<inertial>
 			<origin xyz="-0.29477536 -0.00002361 0.04762554" rpy="0 0 0"/>
@@ -92,16 +74,10 @@
 			<material name="${indy_material}"/>
 		</visual>
-		<collision>
-			<origin xyz="-0.1335 0 -0.075" rpy="${PI/2} 0 -${PI/2}"/>
-			<geometry>
-				<cylinder length="0.267" radius="0.045"/>
-			</geometry>
-		</collision>
-		<collision>
-			<origin xyz="0 0 -0.0375" rpy="0 0 0"/>
-			<geometry>
-				<cylinder length="0.075" radius="0.045"/>
-			</geometry>
-		</collision>
+         <collision>
+            <origin xyz="0 0 0" rpy="0 0 0"/>
+           	<geometry>
+				<mesh filename="package://indy7_description/meshes/collision/Indy7_3.stl"/>
+			</geometry>
+        </collision>
 		<inertial>
 			<origin xyz="-0.16804016 0.00021421 -0.07000383" rpy="0 0 0"/>
@@ -118,22 +94,10 @@
 			<material name="${indy_material}"/>
 		</visual>
-		<collision>
-			<origin xyz="0 -0.057 0.083" rpy="${PI/2} 0 0"/>
-			<geometry>
-				<cylinder length="0.114" radius="0.045"/>
-			</geometry>
-		</collision>
-		<collision>
-			<origin xyz="0 -0.057 0.083" rpy="${PI/2} 0 0"/>
-			<geometry>
-				<cylinder length="0.114" radius="0.045"/>
-			</geometry>
-		</collision>
-		<collision>
-			<origin xyz="0 0 0.0415" rpy="0 0 0"/>
-			<geometry>
-				<cylinder length="0.083" radius="0.045"/>
-			</geometry>
-		</collision>
+         <collision>
+            <origin xyz="0 0 0" rpy="0 0 0"/>
+           	<geometry>
+				<mesh filename="package://indy7_description/meshes/collision/Indy7_4.stl"/>
+			</geometry>
+        </collision>
 		<inertial>
 			<origin xyz="-0.00026847 -0.07098440 0.07649128" rpy="0 0 0"/>
@@ -150,16 +114,10 @@
 			<material name="${indy_material}"/>
 		</visual>
-		<collision>
-			<origin xyz="-0.084 0 0.069" rpy="${PI/2} 0 -${PI/2}"/>
-			<geometry>
-				<cylinder length="0.168" radius="0.045"/>
-			</geometry>
-		</collision>
-		<collision>
-			<origin xyz="-0 0 0.0345" rpy="0 0 0"/>
-			<geometry>
-				<cylinder length="0.069" radius="0.045"/>
-			</geometry>
-		</collision>
+         <collision>
+            <origin xyz="0 0 0" rpy="0 0 0"/>
+           	<geometry>
+				<mesh filename="package://indy7_description/meshes/collision/Indy7_5.stl"/>
+			</geometry>
+        </collision>
 		<inertial>
 			<origin xyz="-0.09796232 -0.00023114 0.06445892" rpy="0 0 0"/>
@@ -176,10 +134,10 @@
 			<material name="${indy_material}"/>
 		</visual>
-		<collision>
-			<origin xyz="0 0 0.03" rpy="0 0 0"/>
-			<geometry>
-				<cylinder length="0.06" radius="0.045"/>
-			</geometry>
-		</collision>
+         <collision>
+            <origin xyz="0 0 0" rpy="0 0 0"/>
+           	<geometry>
+				<mesh filename="package://indy7_description/meshes/collision/Indy7_6.stl"/>
+			</geometry>
+        </collision>
 		<inertial>
 			<origin xyz="0.00008147 -0.00046556 0.03079097" rpy="0 0 0"/>

File: indyrp2_description/urdf/indyrp2.xacro (robot description, xacro)
@@ -60,7 +60,7 @@
         </collision>
          <inertial>
-            <origin xyz="-0.19234403 0.05941510 0.15292668" rpy="0 0 0"/>
+            <origin xyz="-0.21209188 -0.00001715 0.07901191" rpy="0 0 0"/>
             <mass value="4.43308185" />
-            <inertia ixx="+0.03742681" iyy="+0.32119654" izz="+0.29396155" ixy="-0.00003176" iyz="-0.00000808" ixz="+0.07906734"/>
+            <inertia ixx="+0.03742681" iyy="+0.32119654" izz="+0.29396155" ixy="+0.00003176" iyz="-0.00000808" ixz="-0.07906734"/>
         </inertial>
     </link>
@@ -80,7 +80,7 @@
         </collision>
          <inertial>
-            <origin xyz="-0.60631468 0.12700778 0.02546394" rpy="0 0 0"/>
+            <origin xyz="0.00003637 0.07143055 0.07746050" rpy="0 0 0"/>
             <mass value="2.87045928" />
-            <inertia ixx="+0.04098160" iyy="+0.02106773" izz="+0.02277477" ixy="+0.00000747" iyz="-0.01817157" ixz="-0.00000916"/>
+            <inertia ixx="+0.04098160" iyy="+0.02106773" izz="+0.02277477" ixy="+0.00000747" iyz="+0.01817157" ixz="+0.00000916"/>
         </inertial>
     </link>
@@ -176,4 +176,5 @@
     	<origin xyz = "+0.00000000 +0.00000000 +0.07720000" rpy = "0 0 0"/>
     	<axis xyz = "0 0 1"/>
+		<limit effort="10" velocity="1" lower="-${175*PI/180}" upper="${175*PI/180}"/>
     </joint>
     <joint name = "joint1" type = "continuous">
@@ -182,4 +183,5 @@
     	<origin xyz = "+0.00000000 -0.10930000 +0.22280000" rpy = "${PI/2} ${PI/2} 0"/>
     	<axis xyz = "0 0 1"/>
+		<limit effort="10" velocity="1" lower="-${175*PI/180}" upper="${175*PI/180}"/>
     </joint>
     <joint name = "joint2" type = "continuous">
@@ -188,4 +190,5 @@
     	<origin xyz = "-0.38400000 +0.00000000 +0.08470000" rpy = "-${PI/2} 0 ${PI/2}"/>
     	<axis xyz = "0 0 1"/>
+		<limit effort="10" velocity="1" lower="-${175*PI/180}" upper="${175*PI/180}"/>
     </joint>
     <joint name = "joint3" type = "continuous">
@@ -194,4 +197,5 @@
     	<origin xyz = "+0.00000000 +0.11530000 +0.06550000" rpy = "${PI/2} ${PI/2} 0"/>
     	<axis xyz = "0 0 1"/>
+		<limit effort="10" velocity="1" lower="-${175*PI/180}" upper="${175*PI/180}"/>
     </joint>
     <joint name = "joint4" type = "continuous">
@@ -200,4 +204,5 @@
     	<origin xyz = "-0.26650000 +0.00000000 -0.07470000" rpy = "-${PI/2} 0 ${PI/2}"/>
     	<axis xyz = "0 0 1"/>
+		<limit effort="10" velocity="1" lower="-${175*PI/180}" upper="${175*PI/180}"/>
     </joint>
     <joint name = "joint5" type = "continuous">
@@ -206,4 +211,5 @@
     	<origin xyz = "+0.00000000 -0.11430000 +0.08350000" rpy = "${PI/2} ${PI/2} 0"/>
     	<axis xyz = "0 0 1"/>
+		<limit effort="10" velocity="1" lower="-${175*PI/180}" upper="${175*PI/180}"/>
     </joint>
     <joint name = "joint6" type = "continuous">
@@ -212,4 +218,5 @@
         <origin xyz = "-0.16800000 +0.00000000 +0.06870000" rpy = "-${PI/2} 0 ${PI/2}"/>
         <axis xyz = "0 0 1"/>
+		<limit effort="10" velocity="1" lower="-${175*PI/180}" upper="${175*PI/180}"/>
     </joint>
     <joint name = "tcp" type = "fixed">
