Commit message: no message

File: indyrp2_v2_description/urdf/indyrp2_v2.xacro (robot description, xacro)
@@ -16,5 +16,5 @@
             <origin xyz="0 0 0" rpy="0 0 0"/>
            	<geometry>
-				<mesh filename="package://indyrp2_v2_description/collision/stl/IndyRP2_v2_0.stl" />
+				<mesh filename="package://indyrp2_v2_description/meshes/collision/IndyRP2_v2_0.stl" />
 			</geometry>
         </collision>
@@ -36,5 +36,5 @@
             <origin xyz="0 0 0" rpy="0 0 0"/>
            	<geometry>
-				<mesh filename="package://indyrp2_v2_description/collision/stl/IndyRP2_v2_1.stl" />
+				<mesh filename="package://indyrp2_v2_description/meshes/collision/IndyRP2_v2_1.stl" />
 			</geometry>
         </collision>
@@ -56,5 +56,5 @@
             <origin xyz="0 0 0" rpy="0 0 0"/>
            	<geometry>
-				<mesh filename="package://indyrp2_v2_description/collision/stl/IndyRP2_v2_2.stl" />
+				<mesh filename="package://indyrp2_v2_description/meshes/collision/IndyRP2_v2_2.stl" />
 			</geometry>
         </collision>
