Commit message: no message

File: indy12_v2_description/urdf/indy12_v2.xacro (robot description, xacro)
@@ -175,5 +175,5 @@
     	<parent link = "link3"/>
     	<child link = "link4"/>
-    	<origin xyz = "+0.00000000 -0.21000000 -0.10595000" rpy = "$-{PI/2} 0 ${PI}"/>
+    	<origin xyz = "+0.00000000 -0.21000000 -0.10595000" rpy = "-${PI/2} 0 ${PI}"/>
     	<axis xyz = "0 0 1"/>
 		<limit effort="10" velocity="1" lower="-${175*PI/180}" upper="${175*PI/180}"/>

File: indyrp2_v2_description/urdf/indyrp2_v2.xacro (robot description, xacro)
@@ -76,5 +76,5 @@
             <origin xyz="0 0 0" rpy="0 0 0"/>
            	<geometry>
-				<mesh filename="package://indyrp2_v2_description/collision/stl/IndyRP2_v2_3.stl" />
+				<mesh filename="package://indyrp2_v2_description/meshes/collision/IndyRP2_v2_3.stl" />
 			</geometry>
         </collision>
@@ -96,5 +96,5 @@
             <origin xyz="0 0 0" rpy="0 0 0"/>
            	<geometry>
-				<mesh filename="package://indyrp2_v2_description/collision/stl/IndyRP2_v2_4.stl" />
+				<mesh filename="package://indyrp2_v2_description/meshes/collision/IndyRP2_v2_4.stl" />
 			</geometry>
         </collision>
@@ -116,5 +116,5 @@
             <origin xyz="0 0 0" rpy="0 0 0"/>
            	<geometry>
-				<mesh filename="package://indyrp2_v2_description/collision/stl/IndyRP2_v2_5.stl" />
+				<mesh filename="package://indyrp2_v2_description/meshes/collision/IndyRP2_v2_5.stl" />
 			</geometry>
         </collision>
@@ -136,5 +136,5 @@
             <origin xyz="0 0 0" rpy="0 0 0"/>
            	<geometry>
-				<mesh filename="package://indyrp2_v2_description/collision/stl/IndyRP2_v2_6.stl" />
+				<mesh filename="package://indyrp2_v2_description/meshes/collision/IndyRP2_v2_6.stl" />
 			</geometry>
         </collision>
@@ -156,5 +156,5 @@
             <origin xyz="0 0 0" rpy="0 0 0"/>
             <geometry>
-				<mesh filename="package://indyrp2_v2_description/collision/stl/IndyRP2_v2_7.stl" />
+				<mesh filename="package://indyrp2_v2_description/meshes/collision/IndyRP2_v2_7.stl" />
             </geometry>
         </collision>
