Commit message: no message

File: indyrp2_description/urdf/indyrp2.xacro (robot description, xacro)
@@ -171,5 +171,5 @@
     	<origin xyz = "0 0 0" rpy = "0 0 0"/>
     </joint>
-    <joint name = "joint0" type = "continuous">
+    <joint name = "joint0" type = "revolute">
     	<parent link = "link0"/>
     	<child link = "link1"/>
@@ -178,5 +178,5 @@
 		<limit effort="10" velocity="1" lower="-${175*PI/180}" upper="${175*PI/180}"/>
     </joint>
-    <joint name = "joint1" type = "continuous">
+    <joint name = "joint1" type = "revolute">
     	<parent link = "link1"/>
     	<child link = "link2"/>
@@ -185,5 +185,5 @@
 		<limit effort="10" velocity="1" lower="-${175*PI/180}" upper="${175*PI/180}"/>
     </joint>
-    <joint name = "joint2" type = "continuous">
+    <joint name = "joint2" type = "revolute">
     	<parent link = "link2"/>
     	<child link = "link3"/>
@@ -192,5 +192,5 @@
 		<limit effort="10" velocity="1" lower="-${175*PI/180}" upper="${175*PI/180}"/>
     </joint>
-    <joint name = "joint3" type = "continuous">
+    <joint name = "joint3" type = "revolute">
     	<parent link = "link3"/>
     	<child link = "link4"/>
@@ -199,5 +199,5 @@
 		<limit effort="10" velocity="1" lower="-${175*PI/180}" upper="${175*PI/180}"/>
     </joint>
-    <joint name = "joint4" type = "continuous">
+    <joint name = "joint4" type = "revolute">
     	<parent link = "link4"/>
     	<child link = "link5"/>
@@ -206,5 +206,5 @@
 		<limit effort="10" velocity="1" lower="-${175*PI/180}" upper="${175*PI/180}"/>
     </joint>
-    <joint name = "joint5" type = "continuous">
+    <joint name = "joint5" type = "revolute">
     	<parent link = "link5"/>
     	<child link = "link6"/>
@@ -213,5 +213,5 @@
 		<limit effort="10" velocity="1" lower="-${175*PI/180}" upper="${175*PI/180}"/>
     </joint>
-    <joint name = "joint6" type = "continuous">
+    <joint name = "joint6" type = "revolute">
         <parent link = "link6"/>
         <child link = "link7"/>
@@ -225,3 +225,73 @@
     	<origin xyz = "0 0 0.06" rpy = "0 0 0"/>
     </joint>
+	<transmission name="tran0">
+		<type>transmission_interface/SimpleTransmission</type>
+		<joint name="joint0">
+			<hardwareInterface>hardware_interface/PositionJointInterface</hardwareInterface>
+		</joint>
+		<actuator name="motor0">
+			<hardwareInterface>hardware_interface/PositionJointInterface</hardwareInterface>
+			<mechanicalReduction>1</mechanicalReduction>
+		</actuator>
+	</transmission>
+	<transmission name="tran1">
+		<type>transmission_interface/SimpleTransmission</type>
+		<joint name="joint1">
+			<hardwareInterface>hardware_interface/PositionJointInterface</hardwareInterface>
+		</joint>
+		<actuator name="motor1">
+			<hardwareInterface>hardware_interface/PositionJointInterface</hardwareInterface>
+			<mechanicalReduction>1</mechanicalReduction>
+		</actuator>
+	</transmission>
+	<transmission name="tran2">
+		<type>transmission_interface/SimpleTransmission</type>
+		<joint name="joint2">
+			<hardwareInterface>hardware_interface/PositionJointInterface</hardwareInterface>
+		</joint>
+		<actuator name="motor2">
+			<hardwareInterface>hardware_interface/PositionJointInterface</hardwareInterface>
+			<mechanicalReduction>1</mechanicalReduction>
+		</actuator>
+	</transmission>
+	<transmission name="tran3">
+		<type>transmission_interface/SimpleTransmission</type>
+		<joint name="joint3">
+			<hardwareInterface>hardware_interface/PositionJointInterface</hardwareInterface>
+		</joint>
+		<actuator name="motor3">
+			<hardwareInterface>hardware_interface/PositionJointInterface</hardwareInterface>
+			<mechanicalReduction>1</mechanicalReduction>
+		</actuator>
+	</transmission>
+	<transmission name="tran4">
+		<type>transmission_interface/SimpleTransmission</type>
+		<joint name="joint4">
+			<hardwareInterface>hardware_interface/PositionJointInterface</hardwareInterface>
+		</joint>
+		<actuator name="motor4">
+			<hardwareInterface>hardware_interface/PositionJointInterface</hardwareInterface>
+			<mechanicalReduction>1</mechanicalReduction>
+		</actuator>
+	</transmission>
+	<transmission name="tran5">
+		<type>transmission_interface/SimpleTransmission</type>
+		<joint name="joint5">
+			<hardwareInterface>hardware_interface/PositionJointInterface</hardwareInterface>
+		</joint>
+		<actuator name="motor5">
+			<hardwareInterface>hardware_interface/PositionJointInterface</hardwareInterface>
+			<mechanicalReduction>1</mechanicalReduction>
+		</actuator>
+	</transmission>
+	<transmission name="tran6">
+		<type>transmission_interface/SimpleTransmission</type>
+		<joint name="joint6">
+			<hardwareInterface>hardware_interface/PositionJointInterface</hardwareInterface>
+		</joint>
+		<actuator name="motor6">
+			<hardwareInterface>hardware_interface/PositionJointInterface</hardwareInterface>
+			<mechanicalReduction>1</mechanicalReduction>
+		</actuator>
+	</transmission>
 </robot>

File: indyrp2_v2_description/urdf/indyrp2_v2.xacro (robot description, xacro)
@@ -171,5 +171,5 @@
     	<origin xyz = "0 0 0" rpy = "0 0 0"/>
     </joint>
-    <joint name = "joint0" type = "continuous">
+    <joint name = "joint0" type = "revolute">
     	<parent link = "link0"/>
     	<child link = "link1"/>
@@ -178,5 +178,5 @@
 		<limit effort="10" velocity="1" lower="-${175*PI/180}" upper="${175*PI/180}"/>
     </joint>
-    <joint name = "joint1" type = "continuous">
+    <joint name = "joint1" type = "revolute">
     	<parent link = "link1"/>
     	<child link = "link2"/>
@@ -185,5 +185,5 @@
 		<limit effort="10" velocity="1" lower="-${175*PI/180}" upper="${175*PI/180}"/>
     </joint>
-    <joint name = "joint2" type = "continuous">
+    <joint name = "joint2" type = "revolute">
     	<parent link = "link2"/>
     	<child link = "link3"/>
@@ -192,5 +192,5 @@
 		<limit effort="10" velocity="1" lower="-${175*PI/180}" upper="${175*PI/180}"/>
     </joint>
-    <joint name = "joint3" type = "continuous">
+    <joint name = "joint3" type = "revolute">
     	<parent link = "link3"/>
     	<child link = "link4"/>
@@ -199,5 +199,5 @@
 		<limit effort="10" velocity="1" lower="-${175*PI/180}" upper="${175*PI/180}"/>
     </joint>
-    <joint name = "joint4" type = "continuous">
+    <joint name = "joint4" type = "revolute">
     	<parent link = "link4"/>
     	<child link = "link5"/>
@@ -206,5 +206,5 @@
 		<limit effort="10" velocity="1" lower="-${175*PI/180}" upper="${175*PI/180}"/>
     </joint>
-    <joint name = "joint5" type = "continuous">
+    <joint name = "joint5" type = "revolute">
     	<parent link = "link5"/>
     	<child link = "link6"/>
@@ -213,5 +213,5 @@
 		<limit effort="10" velocity="1" lower="-${175*PI/180}" upper="${175*PI/180}"/>
     </joint>
-    <joint name = "joint6" type = "continuous">
+    <joint name = "joint6" type = "revolute">
         <parent link = "link6"/>
         <child link = "link7"/>
@@ -225,3 +225,73 @@
     	<origin xyz = "0 0 0.06" rpy = "0 0 0"/>
     </joint>
+	<transmission name="tran0">
+		<type>transmission_interface/SimpleTransmission</type>
+		<joint name="joint0">
+			<hardwareInterface>hardware_interface/PositionJointInterface</hardwareInterface>
+		</joint>
+		<actuator name="motor0">
+			<hardwareInterface>hardware_interface/PositionJointInterface</hardwareInterface>
+			<mechanicalReduction>1</mechanicalReduction>
+		</actuator>
+	</transmission>
+	<transmission name="tran1">
+		<type>transmission_interface/SimpleTransmission</type>
+		<joint name="joint1">
+			<hardwareInterface>hardware_interface/PositionJointInterface</hardwareInterface>
+		</joint>
+		<actuator name="motor1">
+			<hardwareInterface>hardware_interface/PositionJointInterface</hardwareInterface>
+			<mechanicalReduction>1</mechanicalReduction>
+		</actuator>
+	</transmission>
+	<transmission name="tran2">
+		<type>transmission_interface/SimpleTransmission</type>
+		<joint name="joint2">
+			<hardwareInterface>hardware_interface/PositionJointInterface</hardwareInterface>
+		</joint>
+		<actuator name="motor2">
+			<hardwareInterface>hardware_interface/PositionJointInterface</hardwareInterface>
+			<mechanicalReduction>1</mechanicalReduction>
+		</actuator>
+	</transmission>
+	<transmission name="tran3">
+		<type>transmission_interface/SimpleTransmission</type>
+		<joint name="joint3">
+			<hardwareInterface>hardware_interface/PositionJointInterface</hardwareInterface>
+		</joint>
+		<actuator name="motor3">
+			<hardwareInterface>hardware_interface/PositionJointInterface</hardwareInterface>
+			<mechanicalReduction>1</mechanicalReduction>
+		</actuator>
+	</transmission>
+	<transmission name="tran4">
+		<type>transmission_interface/SimpleTransmission</type>
+		<joint name="joint4">
+			<hardwareInterface>hardware_interface/PositionJointInterface</hardwareInterface>
+		</joint>
+		<actuator name="motor4">
+			<hardwareInterface>hardware_interface/PositionJointInterface</hardwareInterface>
+			<mechanicalReduction>1</mechanicalReduction>
+		</actuator>
+	</transmission>
+	<transmission name="tran5">
+		<type>transmission_interface/SimpleTransmission</type>
+		<joint name="joint5">
+			<hardwareInterface>hardware_interface/PositionJointInterface</hardwareInterface>
+		</joint>
+		<actuator name="motor5">
+			<hardwareInterface>hardware_interface/PositionJointInterface</hardwareInterface>
+			<mechanicalReduction>1</mechanicalReduction>
+		</actuator>
+	</transmission>
+	<transmission name="tran6">
+		<type>transmission_interface/SimpleTransmission</type>
+		<joint name="joint6">
+			<hardwareInterface>hardware_interface/PositionJointInterface</hardwareInterface>
+		</joint>
+		<actuator name="motor6">
+			<hardwareInterface>hardware_interface/PositionJointInterface</hardwareInterface>
+			<mechanicalReduction>1</mechanicalReduction>
+		</actuator>
+	</transmission>
 </robot>
