Commit message: rebuild urdf files

File: src/indy_description/urdf_files/icon3.urdf (robot description, URDF)
Before this commit: robot indy, 9 links, 8 joints
Joints:
- joint joint5: origin xyz=0.0685                          0.0                          0.0 rpy=0.0                         1.570796327                         0.0 -> xyz=0.0685                          0.0                          0.0 rpy=1.570796327                         0.0                         1.570796327
- joint tcp: origin xyz=0 0 0.06 rpy=0 0 0 -> xyz=0.0                          0.0                          0.0 rpy=0.0                         0.0                         0.0

File: src/indy_description/urdf_files/icon7l.urdf (robot description, URDF)
Before this commit: robot indy, 9 links, 8 joints
Joints:
- joint joint5: origin xyz=0.0                          0.089                          0.0 rpy=-1.570796327                         0.0                         0.0 -> xyz=0.0                          0.089                          0.0 rpy=1.570796327                         0.0                         3.14159265
- joint tcp: origin xyz=0 0 0.06 rpy=0 0 0 -> xyz=0.0                          0.0                          0.0 rpy=0.0                         0.0                         0.0

File: src/indy_description/urdf_files/indy12.urdf (robot description, URDF)
Before this commit: robot indy, 9 links, 8 joints
Joints:
- joint tcp: origin xyz=0 0 0.06 rpy=0 0 0 -> xyz=0.0                          0.0                          0.06 rpy=0.0                         0.0                         0.0

File: src/indy_description/urdf_files/indy12_v2.urdf (robot description, URDF)
Before this commit: robot indy, 9 links, 8 joints
Joints:
- joint tcp: origin xyz=0 0 0.06 rpy=0 0 0 -> xyz=0.0                          0.0                          0.09 rpy=0.0                         0.0                         0.0

File: src/indy_description/urdf_files/indy7.urdf (robot description, URDF)
Before this commit: robot indy, 9 links, 8 joints
Joints:
- joint tcp: origin xyz=0 0 0.06 rpy=0 0 0 -> xyz=0.0                          0.0                          0.06 rpy=0.0                         0.0                         0.0

File: src/indy_description/urdf_files/indy7_eye.urdf (robot description, URDF)
Before this commit: robot indy, 9 links, 8 joints
Joints:
- joint tcp: origin xyz=0 0 0.06 rpy=0 0 0 -> xyz=0.0                          0.0                          0.06 rpy=0.0                         0.0                         0.0

File: src/indy_description/urdf_files/indy7_v2.urdf (robot description, URDF)
Before this commit: robot indy, 9 links, 8 joints
Joints:
- joint tcp: origin xyz=0 0 0.06 rpy=0 0 0 -> xyz=0.0                          0.0                          0.06 rpy=0.0                         0.0                         0.0

File: src/indy_description/urdf_files/indyrp2.urdf (robot description, URDF)
Before this commit: robot indy, 10 links, 9 joints
Joints:
- joint tcp: origin xyz=0 0 0.06 rpy=0 0 0 -> xyz=0.0                          0.0                          0.06 rpy=0.0                         0.0                         0.0

File: src/indy_description/urdf_files/indyrp2_eye.urdf (robot description, URDF)
Before this commit: robot indy, 10 links, 9 joints
Joints:
- joint tcp: origin xyz=0 0 0.06 rpy=0 0 0 -> xyz=0.0                          0.0                          0.06 rpy=0.0                         0.0                         0.0

File: src/indy_description/urdf_files/indyrp2_v2.urdf (robot description, URDF)
Before this commit: robot indy, 10 links, 9 joints
Joints:
- joint tcp: origin xyz=0 0 0.06 rpy=0 0 0 -> xyz=0.0                          0.0                          0.06 rpy=0.0                         0.0                         0.0

File: src/indy_description/urdf_files/nuri20c.urdf (robot description, URDF)
Before this commit: robot indy, 9 links, 8 joints
Links:
- link link0: mass 0.858186768 -> 10.512390866
- link link1: mass 2.520440484 -> 18.195720206
- link link2: mass 3.1785267 -> 22.845886455
- link link3: mass 1.601379441 -> 7.83830585
- link link4: mass 1.882223023 -> 6.943393986
- link link5: mass 1.507185922 -> 3.229294314
- link link6: mass 0.634034296 -> 1.586348204
Joints:
- joint tcp: origin xyz=0 0 0.06 rpy=0 0 0 -> xyz=0.0                          0.0                          0.04 rpy=0.0                         0.0                         0.0

File: src/indy_description/urdf_files/nuri3s.urdf (robot description, URDF)
Before this commit: robot indy, 9 links, 8 joints
Joints:
- joint tcp: origin xyz=0 0 0.06 rpy=0 0 0 -> xyz=0.0                          0.0                          0.0285 rpy=0.0                         0.0                         0.0

File: src/indy_description/urdf_files/nuri4s.urdf (robot description, URDF)
Before this commit: robot indy, 9 links, 8 joints
Links:
- link link0: mass 0.858186768 -> 2.861045494
- link link1: mass 2.520440484 -> 3.167175036
- link link2: mass 3.1785267 -> 4.29096783
- link link3: mass 1.601379441 -> 2.018198648
Joints:
- joint tcp: origin xyz=0 0 0.06 rpy=0 0 0 -> xyz=0.0                          0.0                          0.0285 rpy=0.0                         0.0                         0.0

File: src/indy_description/urdf_files/nuri7c.urdf (robot description, URDF)
Before this commit: robot indy, 9 links, 8 joints
Links:
- link link0: mass 0.858186768 -> 4.23
- link link1: mass 2.520440484 -> 5.489055681
- link link2: mass 3.1785267 -> 7.28078719
- link link3: mass 1.601379441 -> 2.871921442
- link link4: mass 1.882223023 -> 2.822752725
- link link5: mass 1.507185922 -> 2.340109457
- link link6: mass 0.634034296 -> 1.141750934
Joints:
- joint tcp: origin xyz=0 0 0.06 rpy=0 0 0 -> xyz=0.0                          0.0                          0.054 rpy=0.0                         0.0                         0.0

File: src/indy_description/urdf_files/opti5.urdf (robot description, URDF)
Before this commit: robot indy, 9 links, 8 joints
Joints:
- joint tcp: origin xyz=0 0 0.06 rpy=0 0 0 -> xyz=0.0                          0.0                          0.0605 rpy=0.0                         0.0                         0.0
