Commit message: update parameters

File: src/indy_description/urdf_files/dual_icon3.urdf (robot description, URDF)
Before this commit: robot indy, 20 links, 19 joints
Joints:
- joint left_arm_connect: origin xyz=0.008367                          0.042157                          0.541659 rpy=-1.570796327                         0.0                         -0.261799388 -> xyz=0.011367                          0.042157                          0.541659 rpy=-1.570796327                         0.0                         -0.261799388
- joint right_arm_connect: origin xyz=0.008367                          -0.042157                          0.541659 rpy=1.570796327                         0.0                         0.261799388 -> xyz=0.011367                          -0.042157                          0.541659 rpy=1.570796327                         0.0                         0.261799388

Commit message: update icon joint_2 zero pos

File: src/indy_description/urdf_files/dual_icon3.urdf (robot description, URDF)
Before this commit: robot indy, 20 links, 19 joints
Joints:
- joint left_arm_joint2: limit lower=-1.8849555921538759 upper=2.652900463031381 effort=197.23 velocity=9.16297857297023 -> lower=-3.4557519189487724 upper=1.0821041362364843 effort=197.23 velocity=9.16297857297023; origin xyz=0.0                          0.26                          0.0 rpy=0.0                         0.0                         0.0 -> xyz=0.0                          0.26                          0.0 rpy=0.0                         0.0                         1.570796327
- joint right_arm_joint2: limit lower=-1.8849555921538759 upper=2.652900463031381 effort=197.23 velocity=9.16297857297023 -> lower=-3.4557519189487724 upper=1.0821041362364843 effort=197.23 velocity=9.16297857297023; origin xyz=0.0                          0.26                          0.0 rpy=0.0                         0.0                         0.0 -> xyz=0.0                          0.26                          0.0 rpy=0.0                         0.0                         1.570796327

File: src/indy_description/urdf_files/icon3.urdf (robot description, URDF)
Before this commit: robot indy, 9 links, 8 joints
Joints:
- joint joint2: limit lower=-1.8849555921538759 upper=2.652900463031381 effort=197.23 velocity=9.16297857297023 -> lower=-3.4557519189487724 upper=1.0821041362364843 effort=197.23 velocity=9.16297857297023; origin xyz=0.0                          0.26                          0.0 rpy=0.0                         0.0                         0.0 -> xyz=0.0                          0.26                          0.0 rpy=0.0                         0.0                         1.570796327

File: src/indy_description/urdf_files/icon7l.urdf (robot description, URDF)
Before this commit: robot indy, 9 links, 8 joints
Joints:
- joint joint2: limit lower=-2.0943951023931953 upper=2.722713633111154 effort=197.23 velocity=6.806784082777885 -> lower=-3.6651914291880923 upper=1.1519173063162575 effort=197.23 velocity=6.806784082777885; origin xyz=0.0                          -0.463                          0.0 rpy=0.0                         0.0                         0.0 -> xyz=0.0                          -0.463                          0.0 rpy=0.0                         0.0                         1.570796327
