Commit message: update parameters

File: src/indy_description/urdf_files/nuri30s.urdf (robot description, URDF)
Before this commit: robot indy, 9 links, 8 joints
Links:
- link link1: mass 20.5 -> 30.0
- link link2: mass 43.88 -> 20.0
- link link3: mass 11.9 -> 9.0
- link link4: mass 5.0 -> 8.0
- link link5: mass 5.0 -> 8.0
- link link6: mass 0.9 -> 1.0
