Commit message: update kinematic for indy12_v2

File: src/indy_description/urdf_files/indy12_v2.urdf (robot description, URDF)
Before this commit: robot indy, 9 links, 8 joints
Joints:
- joint joint0: origin xyz=0                          0                          0.083 rpy=0                         0                         0 -> xyz=0                          0                          0.0815 rpy=0                         0                         0
- joint joint1: origin xyz=0                          -0.137                          0.2675 rpy=1.570796327                         -1.570796327                         0 -> xyz=0                          -0.1355                          0.2685 rpy=1.570796327                         -1.570796327                         0
- joint joint2: origin xyz=0.652                          0                          -0.0205 rpy=0                         0                         1.570796327 -> xyz=0.65                          0                          -0.0185 rpy=0                         0                         1.570796327
- joint joint3: origin xyz=0                          -0.21                          -0.10595 rpy=-1.570796327                         0                         3.14159265 -> xyz=0                          -0.187                          -0.1065 rpy=-1.570796327                         0                         3.14159265
- joint joint4: origin xyz=0                          -0.1305                          0.3628 rpy=-1.570796327                         0                         3.14159265 -> xyz=0                          -0.129                          0.363 rpy=-1.570796327                         0                         3.14159265
- joint joint5: origin xyz=0                          -0.075                          0.08 rpy=-1.570796327                         0                         3.14159265 -> xyz=0                          -0.074                          0.0795 rpy=-1.570796327                         0                         3.14159265
- joint tcp: origin xyz=0.0                          0.0                          0.09 rpy=0.0                         0.0                         0.0 -> xyz=0.0                          0.0                          0.085 rpy=0.0                         0.0                         -0.785398

Commit message: update kinematic for indy12_v2

File: src/indy_description/urdf_files/indy12_v2.urdf (robot description, URDF)
Before this commit: robot indy, 9 links, 8 joints
Joints:
- joint joint5: axis 0 0 -1 -> 0 0 1
- joint tcp: origin xyz=0.0                          0.0                          0.085 rpy=0.0                         0.0                         -0.785398 -> xyz=0.0                          0.0                          0.085 rpy=0.0                         0.0                         0.0
