Commit message: fix moveit, add ICoN3, 7L, Nuri3s, 4s, 20c, Opti5, add servo rx tx topic

File: src/indy_description/urdf/indy_macro.xacro (robot description, xacro)
@@ -19,5 +19,26 @@
         <!-- Load configuration data from the provided .yaml files -->
         <xacro:define_initialize visual_parameters_file="${visual_parameters_file}"/>
-        <xacro:property name="indy_material" value="metal_white"/>
+        <!-- <xacro:property name="indy_material" value="metal_white"/> -->
+        <xacro:if value="${ indy_type == 'indy7' or indy_type == 'indy7_v2' or indy_type == 'indyrp2' or
+                            indy_type == 'indyrp2_v2' or indy_type == 'indy12' or indy_type == 'indy12_v2' or
+                            indy_type == 'nuri3s' or indy_type == 'nuri4s' or indy_type == 'nuri7c' or indy_type == 'nuri20c' or indy_type == 'opti5'}">
+            <xacro:property name="material_0" value="indy_white"/>
+            <xacro:property name="material_1" value="indy_white"/>
+            <xacro:property name="material_2" value="indy_white"/>
+            <xacro:property name="material_3" value="indy_white"/>
+            <xacro:property name="material_4" value="indy_white"/>
+            <xacro:property name="material_5" value="indy_white"/>
+            <xacro:property name="material_6" value="indy_white"/>
+            <xacro:property name="material_7" value="indy_white"/>
+        </xacro:if>
+        <xacro:if value="${indy_type == 'icon3' or indy_type == 'icon7l'}">
+            <xacro:property name="material_0" value="icon_grey"/>
+            <xacro:property name="material_1" value="icon_green"/>
+            <xacro:property name="material_2" value="icon_green"/>
+            <xacro:property name="material_3" value="icon_green"/>
+            <xacro:property name="material_4" value="icon_green"/>
+            <xacro:property name="material_5" value="icon_grey"/>
+            <xacro:property name="material_6" value="icon_grey"/>
+        </xacro:if>
         <!-- links -  main serial chain -->
         <xacro:macro name="define_link" params="link_index link_mesh">
@@ -30,5 +51,29 @@
                         <xacro:get_mesh name="${link_mesh}" type="visual"/>
                     </geometry>
-                    <material name="${indy_material}"/>
+                    <!-- <material name="${indy_material}"/> -->
+                    <xacro:if value="${link_index == 'link0'}">
+                        <material name="${material_0}"/>
+                    </xacro:if>
+                    <xacro:if value="${link_index == 'link1'}">
+                        <material name="${material_1}"/>
+                    </xacro:if>
+                    <xacro:if value="${link_index == 'link2'}">
+                        <material name="${material_2}"/>
+                    </xacro:if>
+                    <xacro:if value="${link_index == 'link3'}">
+                        <material name="${material_3}"/>
+                    </xacro:if>
+                    <xacro:if value="${link_index == 'link4'}">
+                        <material name="${material_4}"/>
+                    </xacro:if>
+                    <xacro:if value="${link_index == 'link5'}">
+                        <material name="${material_5}"/>
+                    </xacro:if>
+                    <xacro:if value="${link_index == 'link6'}">
+                        <material name="${material_6}"/>
+                    </xacro:if>
+                    <xacro:if value="${link_index == 'link7'}">
+                        <material name="${material_7}"/>
+                    </xacro:if>
                 </visual>
                 <collision>

File: src/indy_description/urdf/materials.xacro (robot description, xacro)
@@ -1,36 +1,45 @@
 <?xml version="1.0" ?>
 <robot xmlns:xacro="http://www.ros.org/wiki/xacro">
-	<material name="black">
-		<color rgba="0.0 0.0 0.0 1.0"/>
-	</material>
-	<material name="blue">
-		<color rgba="0.0 0.0 0.8 1.0"/>
-	</material>
-	<material name="green">
-		<color rgba="0.0 0.8 0.0 1.0"/>
-	</material>
-	<material name="grey_">
-		<color rgba="0.2 0.2 0.2 1.0"/>
-	</material>
-	<material name="orange">
-		<color rgba="${255/255} ${108/255} ${10/255} 1.0"/>
-	</material>
-	<material name="brown">
-		<color rgba="${222/255} ${207/255} ${195/255} 1.0"/>
-	</material>
-	<material name="red">
-		<color rgba="0.8 0.0 0.0 1.0"/>
-	</material>
-	<material name="white">
-		<color rgba="1.0 1.0 1.0 1.0"/>
-	</material>
-	<material name="metal">
-		<color rgba="0.768627450980392 0.749019607843137 0.729411764705882 1" />
-	</material>
-	<material name="metal_grey">
-		<color rgba="0.501960784313725 0.501960784313725 0.501960784313725 1" />
-	</material>
-	<material name="metal_white">
-		<color rgba="0.866666666666667 0.866666666666667 0.890196078431373 1" />
-	</material>
+    <material name="black">
+        <color rgba="0.0 0.0 0.0 1.0"/>
+    </material>
+    <material name="blue">
+        <color rgba="0.0 0.0 0.8 1.0"/>
+    </material>
+    <material name="green">
+        <color rgba="0.0 0.8 0.0 1.0"/>
+    </material>
+    <material name="icon_green">
+        <color rgba="${152/255} ${198/255} ${98/255} 1.0"/>
+    </material>
+    <material name="icon_grey">
+        <color rgba="${51/255} ${51/255} ${51/255} 1.0"/>
+    </material>
+    <material name="indy_white">
+        <color rgba="${228/255} ${228/255} ${228/255} 1.0"/>
+    </material>
+    <material name="grey">
+        <color rgba="0.2 0.2 0.2 1.0"/>
+    </material>
+    <material name="orange">
+        <color rgba="${255/255} ${108/255} ${10/255} 1.0"/>
+    </material>
+    <material name="brown">
+        <color rgba="${222/255} ${207/255} ${195/255} 1.0"/>
+    </material>
+    <material name="red">
+        <color rgba="0.8 0.0 0.0 1.0"/>
+    </material>
+    <material name="white">
+        <color rgba="1.0 1.0 1.0 1.0"/>
+    </material>
+    <material name="metal">
+        <color rgba="0.768627450980392 0.749019607843137 0.729411764705882 1" />
+    </material>
+    <material name="metal_grey">
+        <color rgba="0.501960784313725 0.501960784313725 0.501960784313725 1" />
+    </material>
+    <material name="metal_white">
+        <color rgba="0.866666666666667 0.866666666666667 0.890196078431373 1" />
+    </material>
 </robot>

Commit message: add tcp position to kinematics

File: src/indy_description/urdf/indy_macro.xacro (robot description, xacro)
@@ -51,5 +51,4 @@
                         <xacro:get_mesh name="${link_mesh}" type="visual"/>
                     </geometry>
-                    <!-- <material name="${indy_material}"/> -->
                     <xacro:if value="${link_index == 'link0'}">
                         <material name="${material_0}"/>
@@ -158,15 +157,33 @@
         <xacro:if value="${indy_type == 'indyrp2' or indy_type == 'indyrp2_v2'}">
             <xacro:define_joint joint_index="joint6" link_1_index="link6" link_2_index="link7"/>
+            <xacro:property name="config_kinematics_parameters" value="${xacro.load_yaml(kinematics_parameters_file)}"/>
+            <xacro:property name="sec_kinematics" value="${config_kinematics_parameters['kinematics']}" />
             <joint name="${prefix}tcp" type="fixed">
                 <parent link="${prefix}link7"/>
                 <child link="${prefix}tcp"/>
-                <origin xyz="0 0 0.06" rpy="0 0 0"/>
+                <!-- <origin xyz="0 0 0.06" rpy="0 0 0"/> -->
+                <origin
+                    xyz="${sec_kinematics['tcp']['x']}
+                        ${sec_kinematics['tcp']['y']}
+                        ${sec_kinematics['tcp']['z']}"
+                    rpy="${sec_kinematics['tcp']['roll']}
+                        ${sec_kinematics['tcp']['pitch']}
+                        ${sec_kinematics['tcp']['yaw']}"/>
             </joint>
         </xacro:if>
         <xacro:unless value="${indy_type == 'indyrp2' or indy_type == 'indyrp2_v2'}">
+            <xacro:property name="config_kinematics_parameters" value="${xacro.load_yaml(kinematics_parameters_file)}"/>
+            <xacro:property name="sec_kinematics" value="${config_kinematics_parameters['kinematics']}" />
             <joint name="${prefix}tcp" type="fixed">
                 <parent link="${prefix}link6"/>
                 <child link="${prefix}tcp"/>
-                <origin xyz="0 0 0.06" rpy="0 0 0"/>
+                <!-- <origin xyz="0 0 0.06" rpy="0 0 0"/> -->
+                <origin
+                    xyz="${sec_kinematics['tcp']['x']}
+                        ${sec_kinematics['tcp']['y']}
+                        ${sec_kinematics['tcp']['z']}"
+                    rpy="${sec_kinematics['tcp']['roll']}
+                        ${sec_kinematics['tcp']['pitch']}
+                        ${sec_kinematics['tcp']['yaw']}"/>
             </joint>
         </xacro:unless>
