Commit message: add dual icon3

File: src/indy_description/urdf/indy_transmissions.xacro (robot description, xacro)
@@ -13,14 +13,18 @@
             </transmission>
         </xacro:macro>
-        <xacro:define_transmission tran="tran0" joint="joint0" motor="motor0"/>
-        <xacro:define_transmission tran="tran1" joint="joint1" motor="motor1"/>
-        <xacro:define_transmission tran="tran2" joint="joint2" motor="motor2"/>
-        <xacro:define_transmission tran="tran3" joint="joint3" motor="motor3"/>
-        <xacro:define_transmission tran="tran4" joint="joint4" motor="motor4"/>
-        <xacro:define_transmission tran="tran5" joint="joint5" motor="motor5"/>
-        <!--indyrp2 with 7 DOF-->
-        <xacro:if value="${indy_type == 'indyrp2' or indy_type == 'indyrp2_v2'}">
-            <xacro:define_transmission tran="tran6" joint="joint6" motor="motor6"/>
+        <xacro:if value="${indy_type == 'dual_icon3'}">
         </xacro:if>
+        <xacro:unless value="${indy_type == 'dual_icon3'}">
+            <xacro:define_transmission tran="tran0" joint="joint0" motor="motor0"/>
+            <xacro:define_transmission tran="tran1" joint="joint1" motor="motor1"/>
+            <xacro:define_transmission tran="tran2" joint="joint2" motor="motor2"/>
+            <xacro:define_transmission tran="tran3" joint="joint3" motor="motor3"/>
+            <xacro:define_transmission tran="tran4" joint="joint4" motor="motor4"/>
+            <xacro:define_transmission tran="tran5" joint="joint5" motor="motor5"/>
+            <!--indyrp2 with 7 DOF-->
+            <xacro:if value="${indy_type == 'indyrp2' or indy_type == 'indyrp2_v2'}">
+                <xacro:define_transmission tran="tran6" joint="joint6" motor="motor6"/>
+            </xacro:if>
+        </xacro:unless>
     </xacro:macro>
 </robot>
