Commit message: rename to nuri30s, update dynamic parameters

File: src/indy_description/urdf/indy_macro.xacro (robot description, xacro)
@@ -22,5 +22,5 @@
                             indy_type == 'indyrp2_v2' or indy_type == 'indy12' or indy_type == 'indy12_v2' or
                             indy_type == 'nuri3s' or indy_type == 'nuri4s' or indy_type == 'nuri7c' or
-                            indy_type == 'nuri20c' or indy_type == 'nuri35c' or indy_type == 'opti5'}">
+                            indy_type == 'nuri20c' or indy_type == 'nuri30s' or indy_type == 'opti5'}">
             <xacro:property name="material_0" value="indy_white"/>
             <xacro:property name="material_1" value="indy_white"/>

File: src/indy_description/urdf_files/nuri30s.urdf (robot description, URDF)
Before this commit: robot indy, 9 links, 8 joints
Links:
- link link1: mass 30.0 -> 20.5
- link link2: mass 20.0 -> 43.88
- link link3: mass 9.0 -> 11.9
- link link4: mass 8.0 -> 5.0
- link link5: mass 8.0 -> 5.0
- link link6: mass 1.0 -> 0.9

Commit message: update indy7_v3, indyrp2_v2, indy12

File: src/indy_description/urdf/indy_macro.xacro (robot description, xacro)
@@ -19,5 +19,5 @@
         <!-- Load configuration data from the provided .yaml files -->
         <xacro:define_initialize visual_parameters_file="${visual_parameters_file}"/>
-        <xacro:if value="${ indy_type == 'indy7' or indy_type == 'indy7_v2' or indy_type == 'indyrp2' or
+        <xacro:if value="${ indy_type == 'indy7' or indy_type == 'indy7_v2' or indy_type == 'indy7_v3' or indy_type == 'indyrp2' or
                             indy_type == 'indyrp2_v2' or indy_type == 'indy12' or indy_type == 'indy12_v2' or
                             indy_type == 'nuri3s' or indy_type == 'nuri4s' or indy_type == 'nuri7c' or

File: src/indy_description/urdf_files/ar5_left.urdf (robot description, URDF)
Before this commit: robot indy, 9 links, 8 joints
Links:
- added link link7, mass 0.38254932; collision mesh filename=file:///home/user/indy-ros/src/indy_description/meshes/ar5_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; visual mesh filename=file:///home/user/indy-ros/src/indy_description/meshes/ar5_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
- link link0: mass 1.66957888 -> 1.6703078; geometry collision mesh filename=file:///home/user/indy-ros/src/indy_description/meshes/ar5_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; visual mesh filename=file:///home/user/indy-ros/src/indy_description/meshes/ar5_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
- link link1: mass 11.43955917 -> 11.44444535; geometry collision mesh filename=file:///home/user/indy-ros/src/indy_description/meshes/ar5_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; visual mesh filename=file:///home/user/indy-ros/src/indy_description/meshes/ar5_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
- link link2: mass 6.11383823 -> 4.43308185; geometry collision mesh filename=file:///home/user/indy-ros/src/indy_description/meshes/ar5_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; visual mesh filename=file:///home/user/indy-ros/src/indy_description/meshes/ar5_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
- link link3: mass 2.68211719 -> 2.87045928; geometry collision mesh filename=file:///home/user/indy-ros/src/indy_description/meshes/ar5_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; visual mesh filename=file:///home/user/indy-ros/src/indy_description/meshes/ar5_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
- link link4: mass 2.12830848 -> 2.68206064; geometry collision mesh filename=file:///home/user/indy-ros/src/indy_description/meshes/ar5_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; visual mesh filename=file:///home/user/indy-ros/src/indy_description/meshes/ar5_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
- link link5: mass 2.32413397 -> 2.12987371; geometry collision mesh filename=file:///home/user/indy-ros/src/indy_description/meshes/ar5_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; visual mesh filename=file:///home/user/indy-ros/src/indy_description/meshes/ar5_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
- link link6: mass 0.39652271 -> 2.22412271; geometry collision mesh filename=file:///home/user/indy-ros/src/indy_description/meshes/ar5_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; visual mesh filename=file:///home/user/indy-ros/src/indy_description/meshes/ar5_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
Joints:
- added joint joint6: type revolute, parent link6, child link7, origin xyz=0                          0.1245                          -0.0385 rpy=-1.570796327                         0                         0, axis 0 0 1, limit lower=-3.0543261909900767 upper=3.0543261909900767 effort=79.79 velocity=3.141592653589793
- joint joint0: origin xyz=0                          0                          0.0775 rpy=0                         0                         0 -> xyz=0                          0                          0.1042 rpy=0                         0                         0
- joint joint1: origin xyz=0                          -0.109                          0.222 rpy=1.570796327                         0                         0 -> xyz=0                          -0.05315                          0.0703 rpy=1.570796327                         0                         0
- joint joint2: origin xyz=0                          0.45                          -0.0305 rpy=0                         0                         3.1415926536 -> xyz=0                          0.183                          -0.0529 rpy=-1.570796327                         0                         0
- joint joint3: limit lower=-3.0543261909900767 upper=3.0543261909900767 effort=79.79 velocity=3.141592653589793 -> lower=-3.0543261909900767 upper=3.0543261909900767 effort=197.23 velocity=2.6179938779914944; origin xyz=0                          -0.267                          -0.075 rpy=-1.570796327                         0                         3.1415926536 -> xyz=0.01                          -0.05075                          0.131 rpy=1.570796327                         0                         0
- joint joint4: origin xyz=0                          -0.114                          0.0835 rpy=1.570796327                         0                         0 -> xyz=-0.01                          0.128                          -0.05075 rpy=-1.570796327                         0                         0
- joint joint5: limit lower=-3.7524578917878086 upper=3.7524578917878086 effort=79.79 velocity=3.141592653589793 -> lower=-3.0543261909900767 upper=3.0543261909900767 effort=79.79 velocity=3.141592653589793; origin xyz=0                          0.052                          0.085 rpy=-1.570796327                         0                         0 -> xyz=0                          -0.0385                          0.0465 rpy=1.570796327                         0                         0
- joint tcp: origin xyz=0.0                          0.0                          0.0505 rpy=0.0                         0.0                         0.0 -> xyz=0.0                          0.0                          0.037 rpy=0.0                         0.0                         0.0; parent link6 -> link7

File: src/indy_description/urdf_files/ar5_right.urdf (robot description, URDF)
Before this commit: robot indy, 9 links, 8 joints
Links:
- added link link7, mass 0.38254932; collision mesh filename=file:///home/user/indy-ros/src/indy_description/meshes/ar5_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; visual mesh filename=file:///home/user/indy-ros/src/indy_description/meshes/ar5_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
- link link0: mass 1.66957888 -> 1.6703078; geometry collision mesh filename=file:///home/user/indy-ros/src/indy_description/meshes/ar5_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; visual mesh filename=file:///home/user/indy-ros/src/indy_description/meshes/ar5_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
- link link1: mass 11.43955917 -> 11.44444535; geometry collision mesh filename=file:///home/user/indy-ros/src/indy_description/meshes/ar5_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; visual mesh filename=file:///home/user/indy-ros/src/indy_description/meshes/ar5_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
- link link2: mass 6.11383823 -> 4.43308185; geometry collision mesh filename=file:///home/user/indy-ros/src/indy_description/meshes/ar5_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; visual mesh filename=file:///home/user/indy-ros/src/indy_description/meshes/ar5_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
- link link3: mass 2.68211719 -> 2.87045928; geometry collision mesh filename=file:///home/user/indy-ros/src/indy_description/meshes/ar5_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; visual mesh filename=file:///home/user/indy-ros/src/indy_description/meshes/ar5_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
- link link4: mass 2.12830848 -> 2.68206064; geometry collision mesh filename=file:///home/user/indy-ros/src/indy_description/meshes/ar5_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; visual mesh filename=file:///home/user/indy-ros/src/indy_description/meshes/ar5_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
- link link5: mass 2.32413397 -> 2.12987371; geometry collision mesh filename=file:///home/user/indy-ros/src/indy_description/meshes/ar5_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; visual mesh filename=file:///home/user/indy-ros/src/indy_description/meshes/ar5_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
- link link6: mass 0.39652271 -> 2.22412271; geometry collision mesh filename=file:///home/user/indy-ros/src/indy_description/meshes/ar5_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; visual mesh filename=file:///home/user/indy-ros/src/indy_description/meshes/ar5_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
Joints:
- added joint joint6: type revolute, parent link6, child link7, origin xyz=0                          0.1245                          0.0385 rpy=-1.570796327                         0                         0, axis 0 0 1, limit lower=-3.0543261909900767 upper=3.0543261909900767 effort=79.79 velocity=3.141592653589793
- joint joint0: origin xyz=0                          0                          0.0775 rpy=0                         0                         0 -> xyz=0                          0                          0.1042 rpy=0                         0                         0
- joint joint1: origin xyz=0                          -0.109                          0.222 rpy=1.570796327                         0                         0 -> xyz=0                          0.05315                          0.0703 rpy=1.570796327                         0                         0
- joint joint2: origin xyz=0                          0.45                          -0.0305 rpy=0                         0                         3.1415926536 -> xyz=0                          0.183                          0.0529 rpy=-1.570796327                         0                         0
- joint joint3: limit lower=-3.0543261909900767 upper=3.0543261909900767 effort=79.79 velocity=3.141592653589793 -> lower=-3.0543261909900767 upper=3.0543261909900767 effort=197.23 velocity=2.6179938779914944; origin xyz=0                          -0.267                          -0.075 rpy=-1.570796327                         0                         3.1415926536 -> xyz=0.01                          0.05075                          0.131 rpy=1.570796327                         0                         0
- joint joint4: origin xyz=0                          -0.114                          0.0835 rpy=1.570796327                         0                         0 -> xyz=-0.01                          0.128                          0.05075 rpy=-1.570796327                         0                         0
- joint joint5: limit lower=-3.7524578917878086 upper=3.7524578917878086 effort=79.79 velocity=3.141592653589793 -> lower=-3.0543261909900767 upper=3.0543261909900767 effort=79.79 velocity=3.141592653589793; origin xyz=0                          0.052                          0.085 rpy=-1.570796327                         0                         0 -> xyz=0                          0.0385                          0.0465 rpy=1.570796327                         0                         0
- joint tcp: origin xyz=0.0                          0.0                          0.0505 rpy=0.0                         0.0                         0.0 -> xyz=0.0                          0.0                          0.037 rpy=0.0                         0.0                         0.0; parent link6 -> link7

File: src/indy_description/urdf_files/icon7l.urdf (robot description, URDF)
Before this commit: robot indy, 9 links, 8 joints
Joints:
- joint joint1: axis 0 0 1 -> 0 0 -1
- joint joint2: axis 0 0 1 -> 0 0 -1
- joint joint4: axis 0 0 1 -> 0 0 -1
- joint joint5: origin xyz=0.0                          0.089                          0.0 rpy=1.570796327                         0.0                         3.14159265 -> xyz=0.0                          0.089                          0.0 rpy=1.570796327                         1.570796327                         3.14159265

File: src/indy_description/urdf_files/indy12.urdf (robot description, URDF)
Before this commit: robot indy, 9 links, 8 joints
Joints:
- joint joint0: origin xyz=0                          0                          0.13 rpy=0                         0                         0 -> xyz=0                          0                          0.1305 rpy=0                         0                         0
- joint joint1: origin xyz=0                          -0.1275                          0.22 rpy=1.570796327                         -1.570796327                         0 -> xyz=0                          -0.128                          0.2195 rpy=1.570796327                         -1.570796327                         0
- joint tcp: origin xyz=0.0                          0.0                          0.06 rpy=0.0                         0.0                         0.0 -> xyz=0.0                          0.0                          0.056 rpy=0.0                         0.0                         0.0

File: src/indy_description/urdf_files/indy7_v3.urdf (robot description, URDF)
Before this commit: robot indy, 9 links, 8 joints
Joints:
- joint joint0: origin xyz=0                          0                          0.0775 rpy=0                         0                         0 -> xyz=0                          0                          0.0785 rpy=0                         0                         0
- joint joint1: origin xyz=0                          -0.109                          0.222 rpy=1.570796327                         0                         0 -> xyz=0                          -0.1105                          0.2215 rpy=3.1415926536                         1.570796327                         1.570796327
- joint joint2: origin xyz=0                          0.45                          -0.0305 rpy=0                         0                         3.1415926536 -> xyz=-0.45                          0                          -0.0335 rpy=0                         0                         0
- joint joint3: origin xyz=0                          -0.267                          -0.075 rpy=-1.570796327                         0                         3.1415926536 -> xyz=-0.2845                          0                          -0.0735 rpy=1.570796327                         0                         -1.570796327
- joint joint4: origin xyz=0                          -0.114                          0.0835 rpy=1.570796327                         0                         0 -> xyz=0                          0.1405                          0.065486 rpy=-1.570796327                         0                         0
- joint joint5: origin xyz=0                          0.052                          0.085 rpy=-1.570796327                         0                         0 -> xyz=0                          -0.050495                          0.058505 rpy=1.570796327                         3.1415926536                         0
- joint tcp: origin xyz=0.0                          0.0                          0.0505 rpy=0.0                         0.0                         0.0 -> xyz=0.0                          0.0                          0.0557 rpy=0.0                         0.0                         0.0

File: src/indy_description/urdf_files/indyrp2_v2.urdf (robot description, URDF)
Before this commit: robot indy, 10 links, 9 joints
Joints:
- joint joint0: origin xyz=0                          0                          0.0775 rpy=0                         0                         0 -> xyz=0                          0                          0.0785 rpy=0                         0                         0
- joint joint1: origin xyz=0                          -0.109                          0.222 rpy=1.570796327                         0                         0 -> xyz=0                          -0.1103                          0.2215 rpy=1.570796327                         0                         0
- joint joint2: origin xyz=0                          0.361                          0.0845 rpy=-1.570796327                         0                         0 -> xyz=0                          0.3605                          0.0832 rpy=-1.570796327                         0                         0
- joint joint3: origin xyz=0                          0.1153                          0.0885 rpy=-1.570796327                         0                         3.1415926536 -> xyz=0                          0.1163                          0.0895 rpy=-1.570796327                         0                         3.1415926536
- joint joint4: origin xyz=0                          -0.267                          -0.075 rpy=-1.570796327                         0                         3.1415926536 -> xyz=0                          -0.2655                          -0.0737 rpy=-1.570796327                         0                         3.1415926536
- joint joint5: origin xyz=0                          -0.114                          0.0835 rpy=1.570796327                         0                         0 -> xyz=0                          -0.1153                          0.0845 rpy=1.570796327                         0                         0
- joint joint6: origin xyz=0                          0.052                          0.085 rpy=-1.570796327                         0                         0 -> xyz=0                          0.052                          0.0837 rpy=-1.570796327                         0                         0
- joint tcp: origin xyz=0.0                          0.0                          0.057 rpy=0.0                         0.0                         0.0 -> xyz=0.0                          0.0                          0.0515 rpy=0.0                         0.0                         0.0

File: src/indy_description/urdf_files/opti5.urdf (robot description, URDF)
Before this commit: robot indy, 9 links, 8 joints
Joints:
- joint tcp: origin xyz=0.0                          0.0                          0.0605 rpy=0.0                         0.0                         0.0 -> xyz=0.0                          0.0                          0.054 rpy=0.0                         0.0                         0.0

Commit message: add indy12v3, nuri12c, update parameters

File: src/indy_description/urdf/indy_macro.xacro (robot description, xacro)
@@ -20,7 +20,7 @@
         <xacro:define_initialize visual_parameters_file="${visual_parameters_file}"/>
         <xacro:if value="${ indy_type == 'indy7' or indy_type == 'indy7_v2' or indy_type == 'indy7_v3' or indy_type == 'indyrp2' or
-                            indy_type == 'indyrp2_v2' or indy_type == 'indy12' or indy_type == 'indy12_v2' or
-                            indy_type == 'nuri3s' or indy_type == 'nuri4s' or indy_type == 'nuri7c' or
-                            indy_type == 'nuri20c' or indy_type == 'nuri30s' or indy_type == 'opti5'}">
+                            indy_type == 'indyrp2_v2' or indy_type == 'indy12' or indy_type == 'indy12_v2' or indy_type == 'indy12_v3' or
+                            indy_type == 'nuri3s' or indy_type == 'nuri4s' or indy_type == 'nuri7c' or indy_type == 'nuri12c' or
+                            indy_type == 'nuri20c' or indy_type == 'nuri30' or indy_type == 'opti5'}">
             <xacro:property name="material_0" value="indy_white"/>
             <xacro:property name="material_1" value="indy_white"/>
@@ -37,6 +37,9 @@
                 <xacro:property name="sec_inertia_parameters" value="${config_physical_parameters['inertia_parameters']}" />
                 <xacro:if value="${visual_name != ''}">
+                    <xacro:property name="visual_link_entry" value="${sec_mesh_files[visual_name]}"/>
+                    <xacro:property name="visual_origin_xyz" value="${visual_link_entry['visual_origin']['xyz'] if 'visual_origin' in visual_link_entry else '0 0 0'}"/>
+                    <xacro:property name="visual_origin_rpy" value="${visual_link_entry['visual_origin']['rpy'] if 'visual_origin' in visual_link_entry else '0 0 0'}"/>
                     <visual>
-                        <origin xyz="0 0 0" rpy="0 0 0"/>
+                        <origin xyz="${visual_origin_xyz}" rpy="${visual_origin_rpy}"/>
                         <geometry>
                             <xacro:get_mesh name="${visual_name}" type="visual"/>
@@ -45,5 +48,5 @@
                     </visual>
                     <collision>
-                        <origin xyz="0 0 0" rpy="0 0 0"/>
+                        <origin xyz="${visual_origin_xyz}" rpy="${visual_origin_rpy}"/>
                         <geometry>
                             <xacro:get_mesh name="${visual_name}" type="collision"/>

File: src/indy_description/urdf_files/indy12_v2.urdf (robot description, URDF)
Before this commit: robot indy, 9 links, 8 joints
Links:
- link link2: mass 13.86898329 -> 14.27904794
