Commit message: add axes config files

File: src/indy_description/urdf/indy.urdf.xacro (robot description, xacro)
@@ -12,4 +12,5 @@
   <xacro:arg name="physical_params" default="$(find indy_description)/urdf/config/$(arg indy_type)/physical_parameters.yaml"/>
   <xacro:arg name="visual_params" default="$(find indy_description)/urdf/config/$(arg indy_type)/visual_parameters.yaml"/>
+  <xacro:arg name="joint_axes_params" default="$(find indy_description)/urdf/config/$(arg indy_type)/joint_axes.yaml"/>
   <xacro:arg name="transmission_hw_interface" default="hardware_interface/PositionJointInterface"/>
   <link name="world" />
@@ -24,4 +25,5 @@
     physical_parameters_file="$(arg physical_params)"
     visual_parameters_file="$(arg visual_params)"
+    joint_axes_parameters_file="$(arg joint_axes_params)"
     transmission_hw_interface="$(arg transmission_hw_interface)"
     >

File: src/indy_description/urdf/indy_macro.xacro (robot description, xacro)
@@ -14,4 +14,5 @@
         physical_parameters_file
         visual_parameters_file
+        joint_axes_parameters_file
         transmission_hw_interface:=hardware_interface/PositionJointInterface
         *origin">
@@ -118,6 +119,8 @@
             <xacro:property name="config_joint_limit_parameters" value="${xacro.load_yaml(joint_limits_parameters_file)}"/>
             <xacro:property name="config_kinematics_parameters" value="${xacro.load_yaml(kinematics_parameters_file)}"/>
+            <xacro:property name="config_joint_axes_parameters" value="${xacro.load_yaml(joint_axes_parameters_file)}"/>
             <xacro:property name="sec_kinematics" value="${config_kinematics_parameters['kinematics']}" />
             <xacro:property name="sec_limits" value="${config_joint_limit_parameters['joint_limits']}"/>
+            <xacro:property name="sec_joint_axes" value="${config_joint_axes_parameters['joint_axes']}" />
             <joint name="${prefix}${joint_index}" type="${joint_type}">
                 <parent link="${prefix}${parent_link}"/>
@@ -131,5 +134,11 @@
                         ${sec_kinematics[joint_index]['yaw']}"/>
                 <xacro:if value="${joint_type == 'revolute' or joint_type == 'continuous'}">
-                    <axis xyz="0 0 1"/>
+                    <!-- Use configurable axis if available, fallback to default [0,0,1] -->
+                    <xacro:if value="${joint_index in sec_joint_axes}">
+                        <axis xyz="${sec_joint_axes[joint_index][0]} ${sec_joint_axes[joint_index][1]} ${sec_joint_axes[joint_index][2]}"/>
+                    </xacro:if>
+                    <xacro:unless value="${joint_index in sec_joint_axes}">
+                        <axis xyz="0 0 1"/>
+                    </xacro:unless>
                     <dynamics damping="0.1" friction="10.0"/>
                 </xacro:if>

File: src/indy_description/urdf_files/icon3.urdf (robot description, URDF)
Before this commit: robot indy, 9 links, 8 joints
Joints:
- joint joint1: axis 0 0 1 -> 0 0 -1
- joint joint2: axis 0 0 1 -> 0 0 -1
- joint joint4: axis 0 0 1 -> 0 0 -1

File: src/indy_description/urdf_files/indy12_v2.urdf (robot description, URDF)
Before this commit: robot indy, 9 links, 8 joints
Joints:
- joint joint5: axis 0 0 1 -> 0 0 -1

File: src/indy_description/urdf_files/indy7_v2.urdf (robot description, URDF)
Before this commit: robot indy, 9 links, 8 joints
Joints:
- joint tcp: origin xyz=0.0                          0.0                          0.06 rpy=0.0                         0.0                         0.0 -> xyz=0.0                          0.0                          0.057 rpy=0.0                         0.0                         0.0

File: src/indy_description/urdf_files/indyrp2_v2.urdf (robot description, URDF)
Before this commit: robot indy, 10 links, 9 joints
Joints:
- joint tcp: origin xyz=0.0                          0.0                          0.06 rpy=0.0                         0.0                         0.0 -> xyz=0.0                          0.0                          0.057 rpy=0.0                         0.0                         0.0

File: src/indy_description/urdf_files/nuri20c.urdf (robot description, URDF)
Before this commit: robot indy, 9 links, 8 joints
Joints:
- joint joint1: axis 0 0 1 -> 0 0 -1

File: src/indy_description/urdf_files/nuri3s.urdf (robot description, URDF)
Before this commit: robot indy, 9 links, 8 joints
Joints:
- joint joint1: axis 0 0 1 -> 0 0 -1

File: src/indy_description/urdf_files/nuri4s.urdf (robot description, URDF)
Before this commit: robot indy, 9 links, 8 joints
Joints:
- joint joint1: axis 0 0 1 -> 0 0 -1
- joint joint2: axis 0 0 1 -> 0 0 -1
- joint joint4: axis 0 0 1 -> 0 0 -1

File: src/indy_description/urdf_files/nuri7c.urdf (robot description, URDF)
Before this commit: robot indy, 9 links, 8 joints
Joints:
- joint joint1: axis 0 0 1 -> 0 0 -1
