Commit message: add nuri50

File: src/indy_description/urdf/indy.urdf.xacro (robot description, xacro)
@@ -7,10 +7,13 @@
   <xacro:arg name="indy_eye" 	  default="false"/>
   <xacro:arg name="sim_gazebo"  default="false"/>
+  <!-- NURI5s shares the NURI4s geometry and joint parameters. -->
+  <xacro:property name="requested_indy_type" value="$(arg indy_type)"/>
+  <xacro:property name="config_indy_type" value="${'nuri4s' if requested_indy_type == 'nuri5s' else requested_indy_type}"/>
   <!-- parameters -->
-  <xacro:arg name="joint_limit_params" default="$(find indy_description)/urdf/config/$(arg indy_type)/joint_limits.yaml"/>
-  <xacro:arg name="kinematics_params" default="$(find indy_description)/urdf/config/$(arg indy_type)/kinematics.yaml"/>
-  <xacro:arg name="physical_params" default="$(find indy_description)/urdf/config/$(arg indy_type)/physical_parameters.yaml"/>
-  <xacro:arg name="visual_params" default="$(find indy_description)/urdf/config/$(arg indy_type)/visual_parameters.yaml"/>
-  <xacro:arg name="joint_axes_params" default="$(find indy_description)/urdf/config/$(arg indy_type)/joint_axes.yaml"/>
+  <xacro:arg name="joint_limit_params" default="$(find indy_description)/urdf/config/${config_indy_type}/joint_limits.yaml"/>
+  <xacro:arg name="kinematics_params" default="$(find indy_description)/urdf/config/${config_indy_type}/kinematics.yaml"/>
+  <xacro:arg name="physical_params" default="$(find indy_description)/urdf/config/${config_indy_type}/physical_parameters.yaml"/>
+  <xacro:arg name="visual_params" default="$(find indy_description)/urdf/config/${config_indy_type}/visual_parameters.yaml"/>
+  <xacro:arg name="joint_axes_params" default="$(find indy_description)/urdf/config/${config_indy_type}/joint_axes.yaml"/>
   <xacro:arg name="transmission_hw_interface" default="hardware_interface/PositionJointInterface"/>
   <link name="world" />

File: src/indy_description/urdf/indy_macro.xacro (robot description, xacro)
@@ -22,5 +22,6 @@
                             indy_type == 'indyrp2_v2' or indy_type == 'indy12' or indy_type == 'indy12_v2' or indy_type == 'indy12_v3' or
                             indy_type == 'nuri3s' or indy_type == 'nuri4s' or indy_type == 'nuri7c' or indy_type == 'nuri12c' or
-                            indy_type == 'nuri20c' or indy_type == 'nuri30' or indy_type == 'opti5'}">
+                            indy_type == 'nuri20c' or indy_type == 'nuri30' or indy_type == 'nuri50' or
+                            indy_type == 'nuri5s' or indy_type == 'nuri5sdual' or indy_type == 'opti5' or indy_type == 'opti3'}">
             <xacro:property name="material_0" value="indy_white"/>
             <xacro:property name="material_1" value="indy_white"/>
@@ -33,4 +34,5 @@
         <xacro:property name="supports_link6_eye" value="${indy_type == 'indy7' or indy_type == 'indy7_v2' or indy_type == 'indy7_v3' or indy_type == 'indy12_v3'}"/>
         <xacro:property name="supports_link7_eye" value="${indy_type == 'indyrp2' or indy_type == 'indyrp2_v2'}"/>
+        <xacro:property name="is_dual_robot" value="${indy_type == 'dual_icon3' or indy_type == 'nuri5sdual'}"/>
         <!-- links -  main serial chain -->
         <xacro:macro name="define_link" params="link_name physic_name visual_name material gazebo_material">
@@ -73,9 +75,11 @@
             </link>
         </xacro:macro>
-        <xacro:if value="${indy_type == 'dual_icon3'}">
+        <xacro:if value="${is_dual_robot}">
             <!--body-->
             <xacro:define_link link_name="body_base" physic_name="body_base" visual_name="body_base" material="${material_0}" gazebo_material=""/>
+            <xacro:if value="${indy_type == 'dual_icon3'}">
             <xacro:define_link link_name="body_frame" physic_name="body_frame" visual_name="body_frame" material="${material_0}" gazebo_material=""/>
             <xacro:define_link link_name="body_cover" physic_name="body_cover" visual_name="body_cover" material="${material_2}" gazebo_material=""/>
+            </xacro:if>
             <!-- icon3 - left -->
             <xacro:define_link link_name="left_arm_link0" physic_name="left_arm_link0" visual_name="left_arm_link0" material="${material_0}" gazebo_material=""/>
@@ -97,5 +101,5 @@
             <link name="${prefix}right_arm_tcp"/>
         </xacro:if>
-        <xacro:unless value="${indy_type == 'dual_icon3'}">
+        <xacro:unless value="${is_dual_robot}">
             <xacro:define_link link_name="link0" physic_name="link0" visual_name="link0" material="${material_0}" gazebo_material=""/>
             <xacro:define_link link_name="link1" physic_name="link1" visual_name="link1" material="${material_1}" gazebo_material=""/>
@@ -160,5 +164,5 @@
             </joint>
         </xacro:macro>
-        <xacro:if value="${indy_type == 'dual_icon3'}">
+        <xacro:if value="${is_dual_robot}">
             <joint name="global" type="fixed">
                 <origin xyz="0 0 0" rpy="0 0 0"/>
@@ -166,8 +170,14 @@
                 <child link="$(arg prefix)body_base"/>
             </joint>
-            <xacro:define_joint joint_type="revolute" joint_index="base_frame" parent_link="body_base" child_link="body_frame"/>
-            <xacro:define_joint joint_type="fixed" joint_index="frame_cover" parent_link="body_frame" child_link="body_cover"/>
-            <xacro:define_joint joint_type="fixed" joint_index="left_arm_connect" parent_link="body_frame" child_link="left_arm_link0"/>
-            <xacro:define_joint joint_type="fixed" joint_index="right_arm_connect" parent_link="body_frame" child_link="right_arm_link0"/>
+            <xacro:if value="${indy_type == 'dual_icon3'}">
+                <xacro:define_joint joint_type="revolute" joint_index="base_frame" parent_link="body_base" child_link="body_frame"/>
+                <xacro:define_joint joint_type="fixed" joint_index="frame_cover" parent_link="body_frame" child_link="body_cover"/>
+                <xacro:define_joint joint_type="fixed" joint_index="left_arm_connect" parent_link="body_frame" child_link="left_arm_link0"/>
+                <xacro:define_joint joint_type="fixed" joint_index="right_arm_connect" parent_link="body_frame" child_link="right_arm_link0"/>
+            </xacro:if>
+            <xacro:if value="${indy_type == 'nuri5sdual'}">
+                <xacro:define_joint joint_type="fixed" joint_index="left_arm_connect" parent_link="body_base" child_link="left_arm_link0"/>
+                <xacro:define_joint joint_type="fixed" joint_index="right_arm_connect" parent_link="body_base" child_link="right_arm_link0"/>
+            </xacro:if>
             <xacro:define_joint joint_type="revolute" joint_index="left_arm_joint0" parent_link="left_arm_link0" child_link="left_arm_link1"/>
             <xacro:define_joint joint_type="revolute" joint_index="left_arm_joint1" parent_link="left_arm_link1" child_link="left_arm_link2"/>
@@ -185,5 +195,5 @@
             <xacro:define_joint joint_type="fixed"    joint_index="right_arm_tcp" parent_link="right_arm_link6" child_link="right_arm_tcp"/>
         </xacro:if>
-        <xacro:unless value="${indy_type == 'dual_icon3'}">
+        <xacro:unless value="${is_dual_robot}">
             <joint name="global" type="fixed">
                 <origin xyz="0 0 0" rpy="0 0 0"/>

File: src/indy_description/urdf/indy_transmissions.xacro (robot description, xacro)
@@ -13,7 +13,19 @@
             </transmission>
         </xacro:macro>
-        <xacro:if value="${indy_type == 'dual_icon3'}">
+        <xacro:if value="${indy_type == 'nuri5sdual'}">
+            <xacro:define_transmission tran="left_tran0" joint="left_arm_joint0" motor="left_motor0"/>
+            <xacro:define_transmission tran="left_tran1" joint="left_arm_joint1" motor="left_motor1"/>
+            <xacro:define_transmission tran="left_tran2" joint="left_arm_joint2" motor="left_motor2"/>
+            <xacro:define_transmission tran="left_tran3" joint="left_arm_joint3" motor="left_motor3"/>
+            <xacro:define_transmission tran="left_tran4" joint="left_arm_joint4" motor="left_motor4"/>
+            <xacro:define_transmission tran="left_tran5" joint="left_arm_joint5" motor="left_motor5"/>
+            <xacro:define_transmission tran="right_tran0" joint="right_arm_joint0" motor="right_motor0"/>
+            <xacro:define_transmission tran="right_tran1" joint="right_arm_joint1" motor="right_motor1"/>
+            <xacro:define_transmission tran="right_tran2" joint="right_arm_joint2" motor="right_motor2"/>
+            <xacro:define_transmission tran="right_tran3" joint="right_arm_joint3" motor="right_motor3"/>
+            <xacro:define_transmission tran="right_tran4" joint="right_arm_joint4" motor="right_motor4"/>
+            <xacro:define_transmission tran="right_tran5" joint="right_arm_joint5" motor="right_motor5"/>
         </xacro:if>
-        <xacro:unless value="${indy_type == 'dual_icon3'}">
+        <xacro:unless value="${indy_type == 'dual_icon3' or indy_type == 'nuri5sdual'}">
             <xacro:define_transmission tran="tran0" joint="joint0" motor="motor0"/>
             <xacro:define_transmission tran="tran1" joint="joint1" motor="motor1"/>

File: src/indy_moveit/config/indy_macro.srdf.xacro (robot description, xacro)
@@ -6,4 +6,32 @@
     -->
     <xacro:macro name="indy_srdf" params="name prefix indy_type">
+        <xacro:if value="${indy_type == 'nuri5sdual'}">
+            <group name="left_arm">
+                <chain base_link="${prefix}left_arm_link0" tip_link="${prefix}left_arm_tcp"/>
+            </group>
+            <group name="right_arm">
+                <chain base_link="${prefix}right_arm_link0" tip_link="${prefix}right_arm_tcp"/>
+            </group>
+            <group name="dual_arm">
+                <group name="left_arm"/>
+                <group name="right_arm"/>
+            </group>
+            <virtual_joint name="FixedBase" type="fixed" parent_frame="global" child_link="world"/>
+            <disable_collisions link1="${prefix}body_base" link2="${prefix}left_arm_link0" reason="Adjacent"/>
+            <disable_collisions link1="${prefix}body_base" link2="${prefix}right_arm_link0" reason="Adjacent"/>
+            <disable_collisions link1="${prefix}left_arm_link0" link2="${prefix}left_arm_link1" reason="Adjacent"/>
+            <disable_collisions link1="${prefix}left_arm_link1" link2="${prefix}left_arm_link2" reason="Adjacent"/>
+            <disable_collisions link1="${prefix}left_arm_link2" link2="${prefix}left_arm_link3" reason="Adjacent"/>
+            <disable_collisions link1="${prefix}left_arm_link3" link2="${prefix}left_arm_link4" reason="Adjacent"/>
+            <disable_collisions link1="${prefix}left_arm_link4" link2="${prefix}left_arm_link5" reason="Adjacent"/>
+            <disable_collisions link1="${prefix}left_arm_link5" link2="${prefix}left_arm_link6" reason="Adjacent"/>
+            <disable_collisions link1="${prefix}right_arm_link0" link2="${prefix}right_arm_link1" reason="Adjacent"/>
+            <disable_collisions link1="${prefix}right_arm_link1" link2="${prefix}right_arm_link2" reason="Adjacent"/>
+            <disable_collisions link1="${prefix}right_arm_link2" link2="${prefix}right_arm_link3" reason="Adjacent"/>
+            <disable_collisions link1="${prefix}right_arm_link3" link2="${prefix}right_arm_link4" reason="Adjacent"/>
+            <disable_collisions link1="${prefix}right_arm_link4" link2="${prefix}right_arm_link5" reason="Adjacent"/>
+            <disable_collisions link1="${prefix}right_arm_link5" link2="${prefix}right_arm_link6" reason="Adjacent"/>
+        </xacro:if>
+        <xacro:unless value="${indy_type == 'nuri5sdual'}">
         <!--GROUPS - Representation of a set of joints and links. This can be useful for specifying DOF to plan for, defining arms, end effectors, etc-->
         <!--LINKS - When a link is specified, the parent joint of that link (if it exists) is automatically included-->
@@ -82,4 +110,5 @@
             <disable_collisions link1="link4" link2="link6" reason="Never" />
         </xacro:unless>
+        </xacro:unless>
     </xacro:macro>
 </robot>
